File: hardware/kicad/cha/mcu.kicad_sch (KiCad schematic)
At the start: 23 parts, among them J4 microSD, J5 Câble PROG-CHA, SW1 Retour menu

Commit message: FPGA configurés par le RP2350 depuis la carte SD (plus de flash)
- Matériel : flash SPI retirées (4 W25Q32, 12 résistances, 4
  condensateurs). Le bus de liaison arrive sur les broches de
  configuration des iCE40 (LK_SCK -> 70 SCK, LK_IO[0] -> 68 SDI,
  LK_CS_N -> 71 SS), qui redeviennent ces entrées après le démarrage.
  CRESET_N commun aux 4 FPGA, tiré à la masse, piloté par le RP2350
  (GP28) ; câble PROG-CHA en 2 x 7 (CRESET_N + masse). Connecteur 2 x 3
  de secours par FPGA (iceprog -S).
- Firmware : fpga_boot.c (reset commun en mode SPI esclave, envoi des
  SDAES/fpga_*.bin l'un après l'autre, contrôle de CDONE) ; testé sur
  PC (bitstreams reçus à l'identique, FPGA laissés en reset si un
  fichier manque).
- make -C hdl sd : fichiers à copier sur la carte SD.
- PCB : table de placement et références des FPGA mises à jour,
  broches réoptimisées.
Placement-routage des FPGA avec les nouvelles broches : en cours.

Co-Authored-By: Claude Opus 5.5 <noreply@anthropic.com>
Claude-Session: https://claude.ai/code/session_01WKfXP1YJ8otGxZ5dsY6Agh
Parts:
- removed C75: 10u, Capacitor_SMD:C_0805_2012Metric, symbol Device:C
- removed C76: 100n, Capacitor_SMD:C_0603_1608Metric, symbol Device:C
- removed J5: Câble PROG-CHA, Connector_PinHeader_2.54mm:PinHeader_2x06_P2.54mm_Vertical, symbol Connector_Generic:Conn_02x06_Odd_Even
- removed R29, R30, R31, R32, R33, R34: 10k, Resistor_SMD:R_0603_1608Metric, symbol Device:R
- added C73: 10u, Capacitor_SMD:C_0805_2012Metric, symbol Device:C
- added C74: 100n, Capacitor_SMD:C_0603_1608Metric, symbol Device:C
- added J5: Câble PROG-CHA, Connector_PinHeader_2.54mm:PinHeader_2x07_P2.54mm_Vertical, symbol Connector_Generic:Conn_02x07_Odd_Even
- added R13, R14, R15, R16, R17, R18: 33, Resistor_SMD:R_0603_1608Metric, symbol Device:R
- R23, R24, R25, R26, R27, R28: value 33 -> 10k
Connections:
- net +3V3: now also R23.1, R24.1, R25.1, R26.1, R27.1, R28.1, C73.1, C74.1
- net CDONE: now also R23.2, J5.10 (Pin_10)
- net CHA_IO0: now also R19.2; no longer R25.2
- net CHA_IO0_MCU: now also R19.1; no longer R25.1
- net CHA_IO1: now also R20.2; no longer R26.2
- net CHA_IO1_MCU: now also R20.1; no longer R26.1
- net CHA_IO2: now also R21.2; no longer R27.2
- net CHA_IO2_MCU: now also R21.1; no longer R27.1
- net CHA_IO3: now also R22.2; no longer R28.2
- net CHA_IO3_MCU: now also R22.1; no longer R28.1
- net CHA_SCK: now also R18.2; no longer R24.2
- net CHA_SCK_MCU: now also R18.1; no longer R24.1
- net CS_P: now also J5.6 (Pin_6)
- net CS_V: now also J5.7 (Pin_7)
- net GND: now also C73.2, C74.2, J5.11 (Pin_11), J5.12 (Pin_12), J5.14 (Pin_14)
- net LK_IRQ: now also J5.8 (Pin_8)
- net MODE: now also J5.9 (Pin_9)
- net PROG_IO0: now also J5.2 (Pin_2), R14.2; no longer R20.2
- net PROG_IO0_MCU: now also R14.1; no longer R20.1
- net PROG_IO1: now also J5.3 (Pin_3), R15.2; no longer R21.2
- net PROG_IO1_MCU: now also R15.1; no longer R21.1
- net PROG_IO2: now also J5.4 (Pin_4), R16.2; no longer R22.2
- net PROG_IO2_MCU: now also R16.1; no longer R22.1
- net PROG_IO3: now also J5.5 (Pin_5), R17.2; no longer R23.2
- net PROG_IO3_MCU: now also R17.1; no longer R23.1
- net PROG_SCK: now also J5.1 (Pin_1), R13.2; no longer R19.2
- net PROG_SCK_MCU: now also R13.1; no longer R19.1
- net SD_CMD: now also R24.2
- net SD_D0: now also R25.2
- net SD_D1: now also R26.2
- net SD_D2: now also R27.2
- net SD_D3: now also R28.2
- net CRESET_N: now reaches A1.34 (GP28)
- net CRESET_N: now also J5.13 (Pin_13)
- no-connect marks 8 -> 7
