File: hardware/kicad/cha/cha.kicad_sch (KiCad schematic)
At the start: 0 parts

Commit message: Pico 2, microSD et bouton sur la carte PROG ; pistes d'alimentation larges
- La carte PROG est côté avant de la cartouche, composants vers l'avant :
  lecteur microSD et bouton accessibles. Le câble PROG-CHA porte
  désormais le bus de liaison C/SM ; connecteur au même endroit sur les
  deux cartes (x = 172 mm), prêt pour un connecteur carte à carte.
- Sous le Pico : ni piste ni via sur la face composants (pastilles de
  test nues sous le module).
- Classes de réseaux écrites dans le .kicad_pro : +5V et VSYS en 0,5 mm,
  +1V2 en 0,3 mm.
- Broches des FPGA réoptimisées ; contrôle Freerouting sans violation ;
  routage des deux cartes et vérification de timing en cours.

Co-Authored-By: Claude Opus 5.5 <noreply@anthropic.com>
Claude-Session: https://claude.ai/code/session_01WKfXP1YJ8otGxZ5dsY6Agh
Other:
- removed sheet RP2350, carte SD, câble
- added sheet Connecteur et alimentations (suite) (power2.kicad_sch)
Changed lines of the file:
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@@
     (instances
       (project "cha"
-        (path "/c2acc1ad-3350-4022-8990-314ed37b470d"
+        (path "/e0c94673-4de7-4c3d-ae38-3ad172bd9211"
           (page "2")))))
   (sheet
@@
     (instances
       (project "cha"
-        (path "/c2acc1ad-3350-4022-8990-314ed37b470d"
+        (path "/e0c94673-4de7-4c3d-ae38-3ad172bd9211"
           (page "3")))))
   (sheet
@@
     (instances
       (project "cha"
-        (path "/c2acc1ad-3350-4022-8990-314ed37b470d"
+        (path "/e0c94673-4de7-4c3d-ae38-3ad172bd9211"
           (page "4")))))
   (sheet
@@
     (instances
       (project "cha"
-        (path "/c2acc1ad-3350-4022-8990-314ed37b470d"
+        (path "/e0c94673-4de7-4c3d-ae38-3ad172bd9211"
           (page "5")))))
   (sheet
@@
     (instances
       (project "cha"
-        (path "/c2acc1ad-3350-4022-8990-314ed37b470d"
+        (path "/e0c94673-4de7-4c3d-ae38-3ad172bd9211"
           (page "6")))))
   (sheet
@@
     (instances
       (project "cha"
-        (path "/c2acc1ad-3350-4022-8990-314ed37b470d"
+        (path "/e0c94673-4de7-4c3d-ae38-3ad172bd9211"
           (page "7")))))
   (sheet
@@
     (fill
       (color 0 0 0 0.0000))
-    (property "Sheetname" "RP2350, carte SD, câble"
+    (property "Sheetname" "Connecteur et alimentations (suite)"
       (at 152.4 67.88 0)
       (effects
@@
           (size 1.27 1.27))
         (justify left bottom)))
-    (property "Sheetfile" "mcu.kicad_sch"
+    (property "Sheetfile" "power2.kicad_sch"
       (at 152.4 94.58 0)
       (effects
@@
     (instances
       (project "cha"
-        (path "/c2acc1ad-3350-4022-8990-314ed37b470d"
+        (path "/e0c94673-4de7-4c3d-ae38-3ad172bd9211"
           (page "8")))))
   (sheet_instances
