File: hardware/kicad/cha/sdram_c.kicad_sch (KiCad schematic)
At the start: 10 parts, among them U14 AS4C32M16SB-6TIN

Commit message: FPGA configurés par le RP2350 depuis la carte SD (plus de flash)
- Matériel : flash SPI retirées (4 W25Q32, 12 résistances, 4
  condensateurs). Le bus de liaison arrive sur les broches de
  configuration des iCE40 (LK_SCK -> 70 SCK, LK_IO[0] -> 68 SDI,
  LK_CS_N -> 71 SS), qui redeviennent ces entrées après le démarrage.
  CRESET_N commun aux 4 FPGA, tiré à la masse, piloté par le RP2350
  (GP28) ; câble PROG-CHA en 2 x 7 (CRESET_N + masse). Connecteur 2 x 3
  de secours par FPGA (iceprog -S).
- Firmware : fpga_boot.c (reset commun en mode SPI esclave, envoi des
  SDAES/fpga_*.bin l'un après l'autre, contrôle de CDONE) ; testé sur
  PC (bitstreams reçus à l'identique, FPGA laissés en reset si un
  fichier manque).
- make -C hdl sd : fichiers à copier sur la carte SD.
- PCB : table de placement et références des FPGA mises à jour,
  broches réoptimisées.
Placement-routage des FPGA avec les nouvelles broches : en cours.

Co-Authored-By: Claude Opus 5.5 <noreply@anthropic.com>
Claude-Session: https://claude.ai/code/session_01WKfXP1YJ8otGxZ5dsY6Agh
Parts:
- removed C50: 10u, Capacitor_SMD:C_0805_2012Metric, symbol Device:C
- removed R12: 33, Resistor_SMD:R_0603_1608Metric, symbol Device:R
- removed U14: AS4C32M16SB-6TIN, Package_SO:TSOP-II-54_22.2x10.16mm_P0.8mm, symbol Memory_RAM:MT48LC16M16A2TG
- added C42: 100n, Capacitor_SMD:C_0603_1608Metric, symbol Device:C
- added R9: 33, Resistor_SMD:R_0603_1608Metric, symbol Device:R
- added U13: AS4C32M16SB-6TIN, Package_SO:TSOP-II-54_22.2x10.16mm_P0.8mm, symbol Memory_RAM:MT48LC16M16A2TG
- C49: value 100n -> 10u; footprint Capacitor_SMD:C_0603_1608Metric -> Capacitor_SMD:C_0805_2012Metric
Connections:
- net +3V3: now also C42.1, U13.1 (VDD), U13.14 (VDD), U13.27 (VDD), U13.3 (VDDQ), U13.43 (VDDQ), U13.49 (VDDQ), U13.9 (VDDQ)
- net C_SD_A0: now also U13.23 (A0)
- net C_SD_A1: now also U13.24 (A1)
- net C_SD_A10: now also U13.22 (A10)
- net C_SD_A11: now also U13.35 (A11)
- net C_SD_A12: now also U13.36 (A12)
- net C_SD_A2: now also U13.25 (A2)
- net C_SD_A3: now also U13.26 (A3)
- net C_SD_A4: now also U13.29 (A4)
- net C_SD_A5: now also U13.30 (A5)
- net C_SD_A6: now also U13.31 (A6)
- net C_SD_A7: now also U13.32 (A7)
- net C_SD_A8: now also U13.33 (A8)
- net C_SD_A9: now also U13.34 (A9)
- net C_SD_BA0: now also U13.20 (BA0)
- net C_SD_BA1: now also U13.21 (BA1)
- net C_SD_CAS_N: now also U13.17 (~{CAS})
- net C_SD_CKE: now also U13.37 (CKE)
- net C_SD_CLK: now also R9.1
- net C_SD_CLK_R: now also R9.2, U13.38 (CLK)
- net C_SD_CS_N: now also U13.19 (~{CS})
- net C_SD_DQ0: now also U13.2 (DQ0)
- net C_SD_DQ1: now also U13.4 (DQ1)
- net C_SD_DQ10: now also U13.45 (DQ10)
- net C_SD_DQ11: now also U13.47 (DQ11)
- net C_SD_DQ12: now also U13.48 (DQ12)
- net C_SD_DQ13: now also U13.50 (DQ13)
- net C_SD_DQ14: now also U13.51 (DQ14)
- net C_SD_DQ15: now also U13.53 (DQ15)
- net C_SD_DQ2: now also U13.5 (DQ2)
- net C_SD_DQ3: now also U13.7 (DQ3)
- net C_SD_DQ4: now also U13.8 (DQ4)
- net C_SD_DQ5: now also U13.10 (DQ5)
- net C_SD_DQ6: now also U13.11 (DQ6)
- net C_SD_DQ7: now also U13.13 (DQ7)
- net C_SD_DQ8: now also U13.42 (DQ8)
- net C_SD_DQ9: now also U13.44 (DQ9)
- net C_SD_DQM0: now also U13.15 (DQML)
- net C_SD_DQM1: now also U13.39 (DQMH)
- net C_SD_RAS_N: now also U13.18 (~{RAS})
- net C_SD_WE_N: now also U13.16 (~{WE})
- net GND: now also C42.2, U13.12 (VSSQ), U13.28 (VSS), U13.41 (VSS), U13.46 (VSSQ), U13.52 (VSSQ), U13.54 (VSS), U13.6 (VSSQ)
Changed lines of the file:
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@@
     (on_board yes)
     (dnp no)
-    (property "Reference" "U14"
+    (property "Reference" "U13"
       (at 68.58 28.1 0)
       (effects
@@
     (instances
       (project "cha"
-        (path "/935eacec-16fe-43ad-aaac-db4f57d9ae4f/2cf4cddb-efe5-4e2a-8597-3b1983a8c859"
-          (reference "U14")
+        (path "/d4eaa97e-bb7e-46e6-b278-332026c2d879/11475c6b-eba5-4a47-9f0e-275b685a156f"
+          (reference "U13")
           (unit 1)))))
   (global_label "+3V3"
@@
     (on_board yes)
     (dnp no)
-    (property "Reference" "R12"
+    (property "Reference" "R9"
       (at 134.62 29.37 0)
       (effects
@@
     (instances
       (project "cha"
-        (path "/935eacec-16fe-43ad-aaac-db4f57d9ae4f/2cf4cddb-efe5-4e2a-8597-3b1983a8c859"
-          (reference "R12")
+        (path "/d4eaa97e-bb7e-46e6-b278-332026c2d879/11475c6b-eba5-4a47-9f0e-275b685a156f"
+          (reference "R9")
           (unit 1)))))
   (global_label "C_SD_CLK"
@@
     (on_board yes)
     (dnp no)
-    (property "Reference" "C43"
+    (property "Reference" "C42"
       (at 190.5 29.37 0)
       (effects
@@
     (instances
       (project "cha"
-        (path "/935eacec-16fe-43ad-aaac-db4f57d9ae4f/2cf4cddb-efe5-4e2a-8597-3b1983a8c859"
-          (reference "C43")
+        (path "/d4eaa97e-bb7e-46e6-b278-332026c2d879/11475c6b-eba5-4a47-9f0e-275b685a156f"
+          (reference "C42")
           (unit 1)))))
   (global_label "+3V3"
@@
     (on_board yes)
     (dnp no)
-    (property "Reference" "C44"
+    (property "Reference" "C43"
       (at 246.38 29.37 0)
       (effects
@@
     (instances
       (project "cha"
-        (path "/935eacec-16fe-43ad-aaac-db4f57d9ae4f/2cf4cddb-efe5-4e2a-8597-3b1983a8c859"
-          (reference "C44")
+        (path "/d4eaa97e-bb7e-46e6-b278-332026c2d879/11475c6b-eba5-4a47-9f0e-275b685a156f"
+          (reference "C43")
           (unit 1)))))
   (global_label "+3V3"
@@
     (on_board yes)
     (dnp no)
-    (property "Reference" "C45"
+    (property "Reference" "C44"
       (at 299.72 29.37 0)
       (effects
@@
     (instances
       (project "cha"
-        (path "/935eacec-16fe-43ad-aaac-db4f57d9ae4f/2cf4cddb-efe5-4e2a-8597-3b1983a8c859"
-          (reference "C45")
+        (path "/d4eaa97e-bb7e-46e6-b278-332026c2d879/11475c6b-eba5-4a47-9f0e-275b685a156f"
+          (reference "C44")
           (unit 1)))))
   (global_label "+3V3"
@@
     (on_board yes)
     (dnp no)
-    (property "Reference" "C46"
+    (property "Reference" "C45"
       (at 355.6 29.37 0)
       (effects
@@
     (instances
       (project "cha"
-        (path "/935eacec-16fe-43ad-aaac-db4f57d9ae4f/2cf4cddb-efe5-4e2a-8597-3b1983a8c859"
-          (reference "C46")
+        (path "/d4eaa97e-bb7e-46e6-b278-332026c2d879/11475c6b-eba5-4a47-9f0e-275b685a156f"
+          (reference "C45")
           (unit 1)))))
   (global_label "+3V3"
@@
     (on_board yes)
     (dnp no)
-    (property "Reference" "C47"
+    (property "Reference" "C46"
       (at 411.48 29.37 0)
       (effects
@@
     (instances
       (project "cha"
-        (path "/935eacec-16fe-43ad-aaac-db4f57d9ae4f/2cf4cddb-efe5-4e2a-8597-3b1983a8c859"
-          (reference "C47")
+        (path "/d4eaa97e-bb7e-46e6-b278-332026c2d879/11475c6b-eba5-4a47-9f0e-275b685a156f"
+          (reference "C46")
           (unit 1)))))
   (global_label "+3V3"
@@
     (on_board yes)
     (dnp no)
-    (property "Reference" "C48"
+    (property "Reference" "C47"
       (at 464.82 29.37 0)
       (effects
@@
     (instances
       (project "cha"
-        (path "/935eacec-16fe-43ad-aaac-db4f57d9ae4f/2cf4cddb-efe5-4e2a-8597-3b1983a8c859"
-          (reference "C48")
+        (path "/d4eaa97e-bb7e-46e6-b278-332026c2d879/11475c6b-eba5-4a47-9f0e-275b685a156f"
+          (reference "C47")
           (unit 1)))))
   (global_label "+3V3"
@@
     (on_board yes)
     (dnp no)
-    (property "Reference" "C49"
+    (property "Reference" "C48"
       (at 520.7 29.37 0)
       (effects
@@
     (instances
       (project "cha"
-        (path "/935eacec-16fe-43ad-aaac-db4f57d9ae4f/2cf4cddb-efe5-4e2a-8597-3b1983a8c859"
-          (reference "C49")
+        (path "/d4eaa97e-bb7e-46e6-b278-332026c2d879/11475c6b-eba5-4a47-9f0e-275b685a156f"
+          (reference "C48")
           (unit 1)))))
   (global_label "+3V3"
@@
     (on_board yes)
     (dnp no)
-    (property "Reference" "C50"
+    (property "Reference" "C49"
       (at 576.58 29.37 0)
       (effects
@@
     (instances
       (project "cha"
-        (path "/935eacec-16fe-43ad-aaac-db4f57d9ae4f/2cf4cddb-efe5-4e2a-8597-3b1983a8c859"
-          (reference "C50")
+        (path "/d4eaa97e-bb7e-46e6-b278-332026c2d879/11475c6b-eba5-4a47-9f0e-275b685a156f"
+          (reference "C49")
           (unit 1)))))
   (global_label "+3V3"

Commit message: Régulateur 3,3 V à découpage, horloge SDRAM adaptée côté FPGA, U8 en 74AHCT125
- AP63203 (TSOT-23-6, sortie fixe 3,3 V, ~90 %) à la place de
  l'AMS1117 : ~0,15 W de pertes au lieu de ~0,75 W et moins de courant
  tiré sur le 5 V de la console ; L 4,7 µH, Cin 10 µF, Cout 2 x 22 µF.
- Résistance série de 33 ohms de l'horloge SDRAM déclarée avec le FPGA :
  placée à 2,7 mm de sa broche (au lieu de ~30 mm, côté SDRAM).
- CHA : U8 (16244 pour 2 canaux) remplacé par un 74AHCT125.
Cartes replacées, contrôle Freerouting sans violation ; routage des
deux cartes et vérification de timing en cours.

Co-Authored-By: Claude Opus 5.5 <noreply@anthropic.com>
Claude-Session: https://claude.ai/code/session_01WKfXP1YJ8otGxZ5dsY6Agh
Parts:
- removed C42: 100n, Capacitor_SMD:C_0603_1608Metric, symbol Device:C
- removed R9: 33, Resistor_SMD:R_0603_1608Metric, symbol Device:R
- added C50: 10u, Capacitor_SMD:C_0805_2012Metric, symbol Device:C
- C49: value 10u -> 100n; footprint Capacitor_SMD:C_0805_2012Metric -> Capacitor_SMD:C_0603_1608Metric
Connections:
- net +3V3: now also C50.1
- net GND: now also C50.2
Changed lines of the file:
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@@
     (instances
       (project "cha"
-        (path "/e0c94673-4de7-4c3d-ae38-3ad172bd9211/6888ebda-17d6-4344-9bf0-1f13622b6def"
+        (path "/e3e9b29e-cfdd-41d0-b129-236ec434a7fe/81acf1d3-952f-4fad-ac27-3c910137a7cb"
           (reference "U13")
           (unit 1)))))
@@
           (size 1.27 1.27)) hide)))
   (symbol
-    (lib_id "Device:R")
+    (lib_id "Device:C")
     (at 134.62 43.18 0)
     (unit 1)
@@
     (on_board yes)
     (dnp no)
-    (property "Reference" "R9"
+    (property "Reference" "C43"
       (at 134.62 29.37 0)
       (effects
         (font
           (size 1.27 1.27))))
-    (property "Value" "33"
+    (property "Value" "100n"
       (at 134.62 56.99 0)
       (effects
         (font
           (size 1.27 1.27))))
-    (property "Footprint" "Resistor_SMD:R_0603_1608Metric"
+    (property "Footprint" "Capacitor_SMD:C_0603_1608Metric"
       (at 134.62 43.18 0)
       (effects
@@
     (instances
       (project "cha"
-        (path "/e0c94673-4de7-4c3d-ae38-3ad172bd9211/6888ebda-17d6-4344-9bf0-1f13622b6def"
-          (reference "R9")
+        (path "/e3e9b29e-cfdd-41d0-b129-236ec434a7fe/81acf1d3-952f-4fad-ac27-3c910137a7cb"
+          (reference "C43")
           (unit 1)))))
-  (global_label "C_SD_CLK"
+  (global_label "+3V3"
     (shape passive)
     (at 134.62 39.37 90)
@@
         (font
           (size 1.27 1.27)) hide)))
-  (global_label "C_SD_CLK_R"
+  (global_label "GND"
     (shape passive)
     (at 134.62 46.99 270)
@@
     (on_board yes)
     (dnp no)
-    (property "Reference" "C42"
+    (property "Reference" "C44"
       (at 190.5 29.37 0)
       (effects
@@
     (instances
       (project "cha"
-        (path "/e0c94673-4de7-4c3d-ae38-3ad172bd9211/6888ebda-17d6-4344-9bf0-1f13622b6def"
-          (reference "C42")
+        (path "/e3e9b29e-cfdd-41d0-b129-236ec434a7fe/81acf1d3-952f-4fad-ac27-3c910137a7cb"
+          (reference "C44")
           (unit 1)))))
   (global_label "+3V3"
@@
     (on_board yes)
     (dnp no)
-    (property "Reference" "C43"
+    (property "Reference" "C45"
       (at 246.38 29.37 0)
       (effects
@@
     (instances
       (project "cha"
-        (path "/e0c94673-4de7-4c3d-ae38-3ad172bd9211/6888ebda-17d6-4344-9bf0-1f13622b6def"
-          (reference "C43")
+        (path "/e3e9b29e-cfdd-41d0-b129-236ec434a7fe/81acf1d3-952f-4fad-ac27-3c910137a7cb"
+          (reference "C45")
           (unit 1)))))
   (global_label "+3V3"
@@
     (on_board yes)
     (dnp no)
-    (property "Reference" "C44"
+    (property "Reference" "C46"
       (at 299.72 29.37 0)
       (effects
@@
     (instances
       (project "cha"
-        (path "/e0c94673-4de7-4c3d-ae38-3ad172bd9211/6888ebda-17d6-4344-9bf0-1f13622b6def"
-          (reference "C44")
+        (path "/e3e9b29e-cfdd-41d0-b129-236ec434a7fe/81acf1d3-952f-4fad-ac27-3c910137a7cb"
+          (reference "C46")
           (unit 1)))))
   (global_label "+3V3"
@@
     (on_board yes)
     (dnp no)
-    (property "Reference" "C45"
+    (property "Reference" "C47"
       (at 355.6 29.37 0)
       (effects
@@
     (instances
       (project "cha"
-        (path "/e0c94673-4de7-4c3d-ae38-3ad172bd9211/6888ebda-17d6-4344-9bf0-1f13622b6def"
-          (reference "C45")
+        (path "/e3e9b29e-cfdd-41d0-b129-236ec434a7fe/81acf1d3-952f-4fad-ac27-3c910137a7cb"
+          (reference "C47")
           (unit 1)))))
   (global_label "+3V3"
@@
     (on_board yes)
     (dnp no)
-    (property "Reference" "C46"
+    (property "Reference" "C48"
       (at 411.48 29.37 0)
       (effects
@@
     (instances
       (project "cha"
-        (path "/e0c94673-4de7-4c3d-ae38-3ad172bd9211/6888ebda-17d6-4344-9bf0-1f13622b6def"
-          (reference "C46")
+        (path "/e3e9b29e-cfdd-41d0-b129-236ec434a7fe/81acf1d3-952f-4fad-ac27-3c910137a7cb"
+          (reference "C48")
           (unit 1)))))
   (global_label "+3V3"
@@
     (on_board yes)
     (dnp no)
-    (property "Reference" "C47"
+    (property "Reference" "C49"
       (at 464.82 29.37 0)
       (effects
@@
     (instances
       (project "cha"
-        (path "/e0c94673-4de7-4c3d-ae38-3ad172bd9211/6888ebda-17d6-4344-9bf0-1f13622b6def"
-          (reference "C47")
+        (path "/e3e9b29e-cfdd-41d0-b129-236ec434a7fe/81acf1d3-952f-4fad-ac27-3c910137a7cb"
+          (reference "C49")
           (unit 1)))))
   (global_label "+3V3"
@@
     (on_board yes)
     (dnp no)
-    (property "Reference" "C48"
+    (property "Reference" "C50"
       (at 520.7 29.37 0)
       (effects
         (font
           (size 1.27 1.27))))
-    (property "Value" "100n"
+    (property "Value" "10u"
       (at 520.7 56.99 0)
       (effects
         (font
           (size 1.27 1.27))))
-    (property "Footprint" "Capacitor_SMD:C_0603_1608Metric"
+    (property "Footprint" "Capacitor_SMD:C_0805_2012Metric"
       (at 520.7 43.18 0)
       (effects
@@
     (instances
       (project "cha"
-        (path "/e0c94673-4de7-4c3d-ae38-3ad172bd9211/6888ebda-17d6-4344-9bf0-1f13622b6def"
-          (reference "C48")
+        (path "/e3e9b29e-cfdd-41d0-b129-236ec434a7fe/81acf1d3-952f-4fad-ac27-3c910137a7cb"
+          (reference "C50")
           (unit 1)))))
   (global_label "+3V3"
@@
       (effects
         (font
-          (size 1.27 1.27)) hide)))
-  (symbol
-    (lib_id "Device:C")
-    (at 576.58 43.18 0)
-    (unit 1)
-    (in_bom yes)
-    (on_board yes)
-    (dnp no)
-    (property "Reference" "C49"
-      (at 576.58 29.37 0)
-      (effects
-        (font
-          (size 1.27 1.27))))
-    (property "Value" "10u"
-      (at 576.58 56.99 0)
-      (effects
-        (font
-          (size 1.27 1.27))))
-    (property "Footprint" "Capacitor_SMD:C_0805_2012Metric"
-      (at 576.58 43.18 0)
-      (effects
-        (font
-          (size 1.27 1.27)) hide))
-    (property "Datasheet" "~"
-      (at 576.58 43.18 0)
-      (effects
-        (font
-          (size 1.27 1.27)) hide))
-    (pin "1"
-)
-    (pin "2"
-)
-    (instances
-      (project "cha"
-        (path "/e0c94673-4de7-4c3d-ae38-3ad172bd9211/6888ebda-17d6-4344-9bf0-1f13622b6def"
-          (reference "C49")
-          (unit 1)))))
-  (global_label "+3V3"
-    (shape passive)
-    (at 576.58 39.37 90)
-    (fields_autoplaced)
-    (effects
-      (font
-        (size 1.27 1.27))
-      (justify left))
-    (property "Intersheetrefs" "${INTERSHEET_REFS}"
-      (at 576.58 39.37 0)
-      (effects
-        (font
-          (size 1.27 1.27)) hide)))
-  (global_label "GND"
-    (shape passive)
-    (at 576.58 46.99 270)
-    (fields_autoplaced)
-    (effects
-      (font
-        (size 1.27 1.27))
-      (justify right))
-    (property "Intersheetrefs" "${INTERSHEET_REFS}"
-      (at 576.58 46.99 0)
-      (effects
-        (font
