File: hardware/kicad/cha/sram.kicad_sch (KiCad schematic)
At the start: 4 parts, among them U17 IS61WV10248EDBLL-10TLI

Commit message: FPGA configurés par le RP2350 depuis la carte SD (plus de flash)
- Matériel : flash SPI retirées (4 W25Q32, 12 résistances, 4
  condensateurs). Le bus de liaison arrive sur les broches de
  configuration des iCE40 (LK_SCK -> 70 SCK, LK_IO[0] -> 68 SDI,
  LK_CS_N -> 71 SS), qui redeviennent ces entrées après le démarrage.
  CRESET_N commun aux 4 FPGA, tiré à la masse, piloté par le RP2350
  (GP28) ; câble PROG-CHA en 2 x 7 (CRESET_N + masse). Connecteur 2 x 3
  de secours par FPGA (iceprog -S).
- Firmware : fpga_boot.c (reset commun en mode SPI esclave, envoi des
  SDAES/fpga_*.bin l'un après l'autre, contrôle de CDONE) ; testé sur
  PC (bitstreams reçus à l'identique, FPGA laissés en reset si un
  fichier manque).
- make -C hdl sd : fichiers à copier sur la carte SD.
- PCB : table de placement et références des FPGA mises à jour,
  broches réoptimisées.
Placement-routage des FPGA avec les nouvelles broches : en cours.

Co-Authored-By: Claude Opus 5.5 <noreply@anthropic.com>
Claude-Session: https://claude.ai/code/session_01WKfXP1YJ8otGxZ5dsY6Agh
Parts:
- removed C73: 100n, Capacitor_SMD:C_0603_1608Metric, symbol Device:C
- removed C74: 10u, Capacitor_SMD:C_0805_2012Metric, symbol Device:C
- removed U17: IS61WV10248EDBLL-10TLI, Package_SO:TSOP-II-44_10.16x18.41mm_P0.8mm, symbol SDAES:IS61WV10248
- added C70, C71: 100n, Capacitor_SMD:C_0603_1608Metric, symbol Device:C
- added U15: IS61WV10248EDBLL-10TLI, Package_SO:TSOP-II-44_10.16x18.41mm_P0.8mm, symbol SDAES:IS61WV10248
- C72: value 100n -> 10u; footprint Capacitor_SMD:C_0603_1608Metric -> Capacitor_SMD:C_0805_2012Metric
Connections:
- net +3V3: now also C70.1, C71.1, U15.11 (VDD), U15.33 (VDD)
- net GND: now also C70.2, C71.2, U15.12 (GND), U15.34 (GND), U15.8 (~{CE})
- net SR_A0: now also U15.3 (A0)
- net SR_A1: now also U15.4 (A1)
- net SR_A10: now also U15.26 (A10)
- net SR_A11: now also U15.27 (A11)
- net SR_A12: now also U15.28 (A12)
- net SR_A13: now also U15.29 (A13)
- net SR_A14: now also U15.30 (A14)
- net SR_A15: now also U15.38 (A15)
- net SR_A16: now also U15.39 (A16)
- net SR_A17: now also U15.40 (A17)
- net SR_A18: now also U15.41 (A18)
- net SR_A19: now also U15.25 (A19)
- net SR_A2: now also U15.5 (A2)
- net SR_A3: now also U15.6 (A3)
- net SR_A4: now also U15.7 (A4)
- net SR_A5: now also U15.16 (A5)
- net SR_A6: now also U15.17 (A6)
- net SR_A7: now also U15.18 (A7)
- net SR_A8: now also U15.19 (A8)
- net SR_A9: now also U15.20 (A9)
- net SR_D0: now also U15.9 (IO0)
- net SR_D1: now also U15.10 (IO1)
- net SR_D2: now also U15.13 (IO2)
- net SR_D3: now also U15.14 (IO3)
- net SR_D4: now also U15.31 (IO4)
- net SR_D5: now also U15.32 (IO5)
- net SR_D6: now also U15.35 (IO6)
- net SR_D7: now also U15.36 (IO7)
- net SR_OE_N: now also U15.37 (~{OE})
- net SR_WE_N: now also U15.15 (~{WE})
Changed lines of the file:
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@@
     (on_board yes)
     (dnp no)
-    (property "Reference" "U17"
+    (property "Reference" "U15"
       (at 68.58 28.1 0)
       (effects
@@
     (instances
       (project "cha"
-        (path "/935eacec-16fe-43ad-aaac-db4f57d9ae4f/e9c4da38-7b8b-4d49-aec9-3611d11de8d0"
-          (reference "U17")
+        (path "/d4eaa97e-bb7e-46e6-b278-332026c2d879/9b365630-bff1-4b44-ba54-7088aea47d93"
+          (reference "U15")
           (unit 1)))))
   (global_label "SR_A0"
@@
     (on_board yes)
     (dnp no)
-    (property "Reference" "C72"
+    (property "Reference" "C70"
       (at 137.16 29.37 0)
       (effects
@@
     (instances
       (project "cha"
-        (path "/935eacec-16fe-43ad-aaac-db4f57d9ae4f/e9c4da38-7b8b-4d49-aec9-3611d11de8d0"
-          (reference "C72")
+        (path "/d4eaa97e-bb7e-46e6-b278-332026c2d879/9b365630-bff1-4b44-ba54-7088aea47d93"
+          (reference "C70")
           (unit 1)))))
   (global_label "+3V3"
@@
     (on_board yes)
     (dnp no)
-    (property "Reference" "C73"
+    (property "Reference" "C71"
       (at 193.04 29.37 0)
       (effects
@@
     (instances
       (project "cha"
-        (path "/935eacec-16fe-43ad-aaac-db4f57d9ae4f/e9c4da38-7b8b-4d49-aec9-3611d11de8d0"
-          (reference "C73")
+        (path "/d4eaa97e-bb7e-46e6-b278-332026c2d879/9b365630-bff1-4b44-ba54-7088aea47d93"
+          (reference "C71")
           (unit 1)))))
   (global_label "+3V3"
@@
     (on_board yes)
     (dnp no)
-    (property "Reference" "C74"
+    (property "Reference" "C72"
       (at 248.92 29.37 0)
       (effects
@@
     (instances
       (project "cha"
-        (path "/935eacec-16fe-43ad-aaac-db4f57d9ae4f/e9c4da38-7b8b-4d49-aec9-3611d11de8d0"
-          (reference "C74")
+        (path "/d4eaa97e-bb7e-46e6-b278-332026c2d879/9b365630-bff1-4b44-ba54-7088aea47d93"
+          (reference "C72")
           (unit 1)))))
   (global_label "+3V3"

Commit message: Régulateur 3,3 V à découpage, horloge SDRAM adaptée côté FPGA, U8 en 74AHCT125
- AP63203 (TSOT-23-6, sortie fixe 3,3 V, ~90 %) à la place de
  l'AMS1117 : ~0,15 W de pertes au lieu de ~0,75 W et moins de courant
  tiré sur le 5 V de la console ; L 4,7 µH, Cin 10 µF, Cout 2 x 22 µF.
- Résistance série de 33 ohms de l'horloge SDRAM déclarée avec le FPGA :
  placée à 2,7 mm de sa broche (au lieu de ~30 mm, côté SDRAM).
- CHA : U8 (16244 pour 2 canaux) remplacé par un 74AHCT125.
Cartes replacées, contrôle Freerouting sans violation ; routage des
deux cartes et vérification de timing en cours.

Co-Authored-By: Claude Opus 5.5 <noreply@anthropic.com>
Claude-Session: https://claude.ai/code/session_01WKfXP1YJ8otGxZ5dsY6Agh
Parts:
- removed C70: 100n, Capacitor_SMD:C_0603_1608Metric, symbol Device:C
- added C73: 10u, Capacitor_SMD:C_0805_2012Metric, symbol Device:C
- C72: value 10u -> 100n; footprint Capacitor_SMD:C_0805_2012Metric -> Capacitor_SMD:C_0603_1608Metric
Connections:
- net +3V3: now also C73.1
- net GND: now also C73.2
Changed lines of the file:
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@@
     (instances
       (project "cha"
-        (path "/e0c94673-4de7-4c3d-ae38-3ad172bd9211/4dccd2d1-3288-4479-ab73-7341d5d3a8d6"
+        (path "/e3e9b29e-cfdd-41d0-b129-236ec434a7fe/3f81861f-4865-4160-8fbc-b41273b62069"
           (reference "U15")
           (unit 1)))))
@@
     (on_board yes)
     (dnp no)
-    (property "Reference" "C70"
+    (property "Reference" "C71"
       (at 137.16 29.37 0)
       (effects
@@
     (instances
       (project "cha"
-        (path "/e0c94673-4de7-4c3d-ae38-3ad172bd9211/4dccd2d1-3288-4479-ab73-7341d5d3a8d6"
-          (reference "C70")
+        (path "/e3e9b29e-cfdd-41d0-b129-236ec434a7fe/3f81861f-4865-4160-8fbc-b41273b62069"
+          (reference "C71")
           (unit 1)))))
   (global_label "+3V3"
@@
     (on_board yes)
     (dnp no)
-    (property "Reference" "C71"
+    (property "Reference" "C72"
       (at 193.04 29.37 0)
       (effects
@@
     (instances
       (project "cha"
-        (path "/e0c94673-4de7-4c3d-ae38-3ad172bd9211/4dccd2d1-3288-4479-ab73-7341d5d3a8d6"
-          (reference "C71")
+        (path "/e3e9b29e-cfdd-41d0-b129-236ec434a7fe/3f81861f-4865-4160-8fbc-b41273b62069"
+          (reference "C72")
           (unit 1)))))
   (global_label "+3V3"
@@
     (on_board yes)
     (dnp no)
-    (property "Reference" "C72"
+    (property "Reference" "C73"
       (at 248.92 29.37 0)
       (effects
@@
     (instances
       (project "cha"
-        (path "/e0c94673-4de7-4c3d-ae38-3ad172bd9211/4dccd2d1-3288-4479-ab73-7341d5d3a8d6"
-          (reference "C72")
+        (path "/e3e9b29e-cfdd-41d0-b129-236ec434a7fe/3f81861f-4865-4160-8fbc-b41273b62069"
+          (reference "C73")
           (unit 1)))))
   (global_label "+3V3"
