File: hardware/kicad/prog/buffers.kicad_sch (KiCad schematic)
At the start: 21 parts, among them U3 74LVC16244A, U4 74LVC16244A, U5 74LVC16244A, U6 74LVC16245A, U7 74LVC16245A, U8 74AHCT125, U9 74LVC1G07

Commit message: Circuits imprimés 2 couches : placement et affectation des broches FPGA
- hardware/gen/pcb.py : empreintes et réseaux depuis boards.py, contour
  depuis outline.py ; ancres placées (contacts, rangée de tampons, FPGA,
  mémoires ; CHA : Pico au centre, microSD et bouton en haut), passifs
  au plus près de leur broche, masse coulée sur les deux faces.
- --pins : signaux des FPGA affectés aux broches tournées vers leur
  cible en conservant l'ordre circulaire (pins_opt.json, repris par
  fpga_pins.py) ; stable en trois passes.
- boards.py : canaux des tampons triés selon la position des contacts.
- hardware/gen/route.py : export Specctra, Freerouting, relecture de la
  session, DRC.
Placement-routage FPGA avec les nouvelles broches : en cours de
vérification.

Co-Authored-By: Claude Opus 5.5 <noreply@anthropic.com>
Claude-Session: https://claude.ai/code/session_01WKfXP1YJ8otGxZ5dsY6Agh
Connections:
- net A1: now also U5.9 (2Y2); no longer U3.2 (1Y1)
- net A10: now also U4.19 (4Y1); no longer U3.14 (3Y2)
- net A11: now also U4.17 (3Y4); no longer U3.16 (3Y3)
- net A12: now also U4.16 (3Y3); no longer U3.17 (3Y4)
- net A13: now also U4.14 (3Y2); no longer U3.19 (4Y1)
- net A14: now also U4.13 (3Y1); no longer U3.20 (4Y2)
- net A15: now also U4.12 (2Y4); no longer U3.22 (4Y3)
- net A16: now also U4.11 (2Y3); no longer U3.23 (4Y4)
- net A17: now also U4.9 (2Y2); no longer U4.2 (1Y1)
- net A18: now also U4.8 (2Y1); no longer U4.3 (1Y2)
- net A19: now also U4.6 (1Y4); no longer U4.5 (1Y3)
- net A2: now also U5.8 (2Y1); no longer U3.3 (1Y2)
- net A3: now also U5.6 (1Y4); no longer U3.5 (1Y3)
- net A4: now also U5.5 (1Y3); no longer U3.6 (1Y4)
- net A5: now also U5.3 (1Y2); no longer U3.8 (2Y1)
- net A6: now also U5.2 (1Y1); no longer U3.9 (2Y2)
- net A7: now also U4.23 (4Y4); no longer U3.11 (2Y3)
- net A8: now also U4.22 (4Y3); no longer U3.12 (2Y4)
- net A9: now also U4.20 (4Y2); no longer U3.13 (3Y1)
- net AES_A1: now also U5.40 (2A2); no longer U3.47 (1A1)
- net AES_A10: now also U4.30 (4A1); no longer U3.35 (3A2)
- net AES_A11: now also U4.32 (3A4); no longer U3.33 (3A3)
- net AES_A12: now also U4.33 (3A3); no longer U3.32 (3A4)
- net AES_A13: now also U4.35 (3A2); no longer U3.30 (4A1)
- net AES_A14: now also U4.36 (3A1); no longer U3.29 (4A2)
- net AES_A15: now also U4.37 (2A4); no longer U3.27 (4A3)
- net AES_A16: now also U4.38 (2A3); no longer U3.26 (4A4)
- net AES_A17: now also U4.40 (2A2); no longer U4.47 (1A1)
- net AES_A18: now also U4.41 (2A1); no longer U4.46 (1A2)
- net AES_A19: now also U4.43 (1A4); no longer U4.44 (1A3)
- net AES_A2: now also U5.41 (2A1); no longer U3.46 (1A2)
- net AES_A3: now also U5.43 (1A4); no longer U3.44 (1A3)
- net AES_A4: now also U5.44 (1A3); no longer U3.43 (1A4)
- net AES_A5: now also U5.46 (1A2); no longer U3.41 (2A1)
- net AES_A6: now also U5.47 (1A1); no longer U3.40 (2A2)
- net AES_A7: now also U4.26 (4A4); no longer U3.38 (2A3)
- net AES_A8: now also U4.27 (4A3); no longer U3.37 (2A4)
- net AES_A9: now also U4.29 (4A2); no longer U3.36 (3A1)
- net AES_D0: now also U6.23 (B15); no longer U6.2 (B0)
- net AES_D1: now also U6.22 (B14); no longer U6.3 (B1)
- net AES_D10: now also U6.9 (B5); no longer U6.16 (B10)
- net AES_D11: now also U6.8 (B4); no longer U6.17 (B11)
- net AES_D12: now also U6.6 (B3); no longer U6.19 (B12)
- net AES_D13: now also U6.5 (B2); no longer U6.20 (B13)
- net AES_D14: now also U6.3 (B1); no longer U6.22 (B14)
- net AES_D15: now also U6.2 (B0); no longer U6.23 (B15)
- net AES_D2: now also U6.20 (B13); no longer U6.5 (B2)
- net AES_D3: now also U6.19 (B12); no longer U6.6 (B3)
- net AES_D4: now also U6.17 (B11); no longer U6.8 (B4)
- net AES_D5: now also U6.16 (B10); no longer U6.9 (B5)
- net AES_D6: now also U6.14 (B9); no longer U6.11 (B6)
- net AES_D7: now also U6.13 (B8); no longer U6.12 (B7)
- net AES_D8: now also U6.12 (B7); no longer U6.13 (B8)
- net AES_D9: now also U6.11 (B6); no longer U6.14 (B9)
- net AES_PORTOEL: now also U4.47 (1A1); no longer U4.40 (2A2)
- net AES_PORTOEU: now also U4.46 (1A2); no longer U4.41 (2A1)
- net AES_PORTWEL: now also U3.27 (4A3); no longer U4.38 (2A3)
- net AES_PORTWEU: now also U3.26 (4A4); no longer U4.37 (2A4)
- net AES_ROMOE: now also U4.44 (1A3); no longer U4.43 (1A4)
- net AES_SDPA10: now also U3.37 (2A4); no longer U5.44 (1A3)
- net AES_SDPA11: now also U3.40 (2A2); no longer U5.43 (1A4)
- net AES_SDPA8: now also U3.32 (3A4); no longer U5.47 (1A1)
- net AES_SDPA9: now also U3.35 (3A2); no longer U5.46 (1A2)
- net AES_SDPAD0: now also U7.23 (B15); no longer U7.13 (B8)
- net AES_SDPAD1: now also U7.22 (B14); no longer U7.14 (B9)
- net AES_SDPAD2: now also U7.20 (B13); no longer U7.16 (B10)
- net AES_SDPAD3: now also U7.19 (B12); no longer U7.17 (B11)
- net AES_SDPAD4: now also U7.17 (B11); no longer U7.19 (B12)
- net AES_SDPAD5: now also U7.16 (B10); no longer U7.20 (B13)
- net AES_SDPAD6: now also U7.14 (B9); no longer U7.22 (B14)
- net AES_SDPAD7: now also U7.13 (B8); no longer U7.23 (B15)
- net AES_SDPMPX: now also U3.43 (1A4); no longer U5.41 (2A1)
- net AES_SDPOE: now also U3.46 (1A2); no longer U5.40 (2A2)
- net AES_SDRA20: now also U3.33 (3A3); no longer U4.33 (3A3)
- net AES_SDRA21: now also U3.36 (3A1); no longer U4.32 (3A4)
- net AES_SDRA22: now also U3.38 (2A3); no longer U4.30 (4A1)
- net AES_SDRA23: now also U3.41 (2A1); no longer U4.29 (4A2)
- net AES_SDRA8: now also U3.29 (4A2); no longer U4.36 (3A1)
- net AES_SDRA9: now also U3.30 (4A1); no longer U4.35 (3A2)
- net AES_SDRAD0: now also U7.12 (B7); no longer U7.2 (B0)
- net AES_SDRAD1: now also U7.11 (B6); no longer U7.3 (B1)
- net AES_SDRAD2: now also U7.9 (B5); no longer U7.5 (B2)
- net AES_SDRAD3: now also U7.8 (B4); no longer U7.6 (B3)
- net AES_SDRAD4: now also U7.6 (B3); no longer U7.8 (B4)
- net AES_SDRAD5: now also U7.5 (B2); no longer U7.9 (B5)
- net AES_SDRAD6: now also U7.3 (B1); no longer U7.11 (B6)
- net AES_SDRAD7: now also U7.2 (B0); no longer U7.12 (B7)
- net AES_SDRMPX: now also U3.44 (1A3); no longer U4.27 (4A3)
- net AES_SDROE: now also U3.47 (1A1); no longer U4.26 (4A4)
- net D0: now also U6.26 (A15); no longer U6.47 (A0)
- net D1: now also U6.27 (A14); no longer U6.46 (A1)
- net D10: now also U6.40 (A5); no longer U6.33 (A10)
- net D11: now also U6.41 (A4); no longer U6.32 (A11)
- net D12: now also U6.43 (A3); no longer U6.30 (A12)
- net D13: now also U6.44 (A2); no longer U6.29 (A13)
- net D14: now also U6.46 (A1); no longer U6.27 (A14)
- net D15: now also U6.47 (A0); no longer U6.26 (A15)
- net D2: now also U6.29 (A13); no longer U6.44 (A2)
- net D3: now also U6.30 (A12); no longer U6.43 (A3)
- net D4: now also U6.32 (A11); no longer U6.41 (A4)
- net D5: now also U6.33 (A10); no longer U6.40 (A5)
- net D6: now also U6.35 (A9); no longer U6.38 (A6)
- net D7: now also U6.36 (A8); no longer U6.37 (A7)
- net D8: now also U6.37 (A7); no longer U6.36 (A8)
- net D9: now also U6.38 (A6); no longer U6.35 (A9)
- net PORTOEL_N: now also U4.2 (1Y1); no longer U4.9 (2Y2)
- net PORTOEU_N: now also U4.3 (1Y2); no longer U4.8 (2Y1)
- net PORTWEL_N: now also U3.22 (4Y3); no longer U4.11 (2Y3)
- net PORTWEU_N: now also U3.23 (4Y4); no longer U4.12 (2Y4)
- net ROMOE_N: now also U4.5 (1Y3); no longer U4.6 (1Y4)
- net SDPA10: now also U3.12 (2Y4); no longer U5.5 (1Y3)
- net SDPA11: now also U3.9 (2Y2); no longer U5.6 (1Y4)
- net SDPA8: now also U3.17 (3Y4); no longer U5.2 (1Y1)
- net SDPA9: now also U3.14 (3Y2); no longer U5.3 (1Y2)
- net SDPAD0: now also U7.26 (A15); no longer U7.36 (A8)
- net SDPAD1: now also U7.27 (A14); no longer U7.35 (A9)
- net SDPAD2: now also U7.29 (A13); no longer U7.33 (A10)
- net SDPAD3: now also U7.30 (A12); no longer U7.32 (A11)
- net SDPAD4: now also U7.32 (A11); no longer U7.30 (A12)
- net SDPAD5: now also U7.33 (A10); no longer U7.29 (A13)
- net SDPAD6: now also U7.35 (A9); no longer U7.27 (A14)
- net SDPAD7: now also U7.36 (A8); no longer U7.26 (A15)
- net SDPMPX: now also U3.6 (1Y4); no longer U5.8 (2Y1)
- net SDPOE_N: now also U3.3 (1Y2); no longer U5.9 (2Y2)
- net SDRA20: now also U3.16 (3Y3); no longer U4.16 (3Y3)
- net SDRA21: now also U3.13 (3Y1); no longer U4.17 (3Y4)
- net SDRA22: now also U3.11 (2Y3); no longer U4.19 (4Y1)
- net SDRA23: now also U3.8 (2Y1); no longer U4.20 (4Y2)
- net SDRA8: now also U3.20 (4Y2); no longer U4.13 (3Y1)
- net SDRA9: now also U3.19 (4Y1); no longer U4.14 (3Y2)
- net SDRAD0: now also U7.37 (A7); no longer U7.47 (A0)
- net SDRAD1: now also U7.38 (A6); no longer U7.46 (A1)
- net SDRAD2: now also U7.40 (A5); no longer U7.44 (A2)
- net SDRAD3: now also U7.41 (A4); no longer U7.43 (A3)
- net SDRAD4: now also U7.43 (A3); no longer U7.41 (A4)
- net SDRAD5: now also U7.44 (A2); no longer U7.40 (A5)
- net SDRAD6: now also U7.46 (A1); no longer U7.38 (A6)
- net SDRAD7: now also U7.47 (A0); no longer U7.37 (A7)
- net SDRMPX: now also U3.5 (1Y3); no longer U4.22 (4Y3)
- net SDROE_N: now also U3.2 (1Y1); no longer U4.23 (4Y4)

Commit message: Régulateur 3,3 V à découpage, horloge SDRAM adaptée côté FPGA, U8 en 74AHCT125
- AP63203 (TSOT-23-6, sortie fixe 3,3 V, ~90 %) à la place de
  l'AMS1117 : ~0,15 W de pertes au lieu de ~0,75 W et moins de courant
  tiré sur le 5 V de la console ; L 4,7 µH, Cin 10 µF, Cout 2 x 22 µF.
- Résistance série de 33 ohms de l'horloge SDRAM déclarée avec le FPGA :
  placée à 2,7 mm de sa broche (au lieu de ~30 mm, côté SDRAM).
- CHA : U8 (16244 pour 2 canaux) remplacé par un 74AHCT125.
Cartes replacées, contrôle Freerouting sans violation ; routage des
deux cartes et vérification de timing en cours.

Co-Authored-By: Claude Opus 5.5 <noreply@anthropic.com>
Claude-Session: https://claude.ai/code/session_01WKfXP1YJ8otGxZ5dsY6Agh
Parts:
- removed C7, C8: 100n, Capacitor_SMD:C_0603_1608Metric, symbol Device:C
- added C19, C20: 100n, Capacitor_SMD:C_0603_1608Metric, symbol Device:C
Connections:
- net +3V3: now also C17.1, C20.1
- net +5V: now also C19.1; no longer C17.1
- net GND: now also C19.2, C20.2
Changed lines of the file:
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@@
     (instances
       (project "prog"
-        (path "/730f52e2-cd0f-4a48-866b-cc2c9ca510b4/d40f7c6c-10f9-4e55-bf54-58eac98e1c03"
+        (path "/3a034faf-f518-4ff2-b4c3-d71a1132e6ac/148c5e2e-2d42-4944-9524-d6f8f44422c9"
           (reference "U3")
           (unit 1)))))
@@
     (on_board yes)
     (dnp no)
-    (property "Reference" "C7"
+    (property "Reference" "C9"
       (at 134.62 29.37 0)
       (effects
@@
     (instances
       (project "prog"
-        (path "/730f52e2-cd0f-4a48-866b-cc2c9ca510b4/d40f7c6c-10f9-4e55-bf54-58eac98e1c03"
-          (reference "C7")
+        (path "/3a034faf-f518-4ff2-b4c3-d71a1132e6ac/148c5e2e-2d42-4944-9524-d6f8f44422c9"
+          (reference "C9")
           (unit 1)))))
   (global_label "+3V3"
@@
     (on_board yes)
     (dnp no)
-    (property "Reference" "C8"
+    (property "Reference" "C10"
       (at 190.5 29.37 0)
       (effects
@@
     (instances
       (project "prog"
-        (path "/730f52e2-cd0f-4a48-866b-cc2c9ca510b4/d40f7c6c-10f9-4e55-bf54-58eac98e1c03"
-          (reference "C8")
+        (path "/3a034faf-f518-4ff2-b4c3-d71a1132e6ac/148c5e2e-2d42-4944-9524-d6f8f44422c9"
+          (reference "C10")
           (unit 1)))))
   (global_label "+3V3"
@@
     (instances
       (project "prog"
-        (path "/730f52e2-cd0f-4a48-866b-cc2c9ca510b4/d40f7c6c-10f9-4e55-bf54-58eac98e1c03"
+        (path "/3a034faf-f518-4ff2-b4c3-d71a1132e6ac/148c5e2e-2d42-4944-9524-d6f8f44422c9"
           (reference "U4")
           (unit 1)))))
@@
     (on_board yes)
     (dnp no)
-    (property "Reference" "C9"
+    (property "Reference" "C11"
       (at 325.12 29.37 0)
       (effects
@@
     (instances
       (project "prog"
-        (path "/730f52e2-cd0f-4a48-866b-cc2c9ca510b4/d40f7c6c-10f9-4e55-bf54-58eac98e1c03"
-          (reference "C9")
+        (path "/3a034faf-f518-4ff2-b4c3-d71a1132e6ac/148c5e2e-2d42-4944-9524-d6f8f44422c9"
+          (reference "C11")
           (unit 1)))))
   (global_label "+3V3"
@@
     (on_board yes)
     (dnp no)
-    (property "Reference" "C10"
+    (property "Reference" "C12"
       (at 381 29.37 0)
       (effects
@@
     (instances
       (project "prog"
-        (path "/730f52e2-cd0f-4a48-866b-cc2c9ca510b4/d40f7c6c-10f9-4e55-bf54-58eac98e1c03"
-          (reference "C10")
+        (path "/3a034faf-f518-4ff2-b4c3-d71a1132e6ac/148c5e2e-2d42-4944-9524-d6f8f44422c9"
+          (reference "C12")
           (unit 1)))))
   (global_label "+3V3"
@@
     (instances
       (project "prog"
-        (path "/730f52e2-cd0f-4a48-866b-cc2c9ca510b4/d40f7c6c-10f9-4e55-bf54-58eac98e1c03"
+        (path "/3a034faf-f518-4ff2-b4c3-d71a1132e6ac/148c5e2e-2d42-4944-9524-d6f8f44422c9"
           (reference "U5")
           (unit 1)))))
@@
     (on_board yes)
     (dnp no)
-    (property "Reference" "C11"
+    (property "Reference" "C13"
       (at 515.62 29.37 0)
       (effects
@@
     (instances
       (project "prog"
-        (path "/730f52e2-cd0f-4a48-866b-cc2c9ca510b4/d40f7c6c-10f9-4e55-bf54-58eac98e1c03"
-          (reference "C11")
+        (path "/3a034faf-f518-4ff2-b4c3-d71a1132e6ac/148c5e2e-2d42-4944-9524-d6f8f44422c9"
+          (reference "C13")
           (unit 1)))))
   (global_label "+3V3"
@@
     (on_board yes)
     (dnp no)
-    (property "Reference" "C12"
+    (property "Reference" "C14"
       (at 571.5 29.37 0)
       (effects
@@
     (instances
       (project "prog"
-        (path "/730f52e2-cd0f-4a48-866b-cc2c9ca510b4/d40f7c6c-10f9-4e55-bf54-58eac98e1c03"
-          (reference "C12")
+        (path "/3a034faf-f518-4ff2-b4c3-d71a1132e6ac/148c5e2e-2d42-4944-9524-d6f8f44422c9"
+          (reference "C14")
           (unit 1)))))
   (global_label "+3V3"
@@
     (instances
       (project "prog"
-        (path "/730f52e2-cd0f-4a48-866b-cc2c9ca510b4/d40f7c6c-10f9-4e55-bf54-58eac98e1c03"
+        (path "/3a034faf-f518-4ff2-b4c3-d71a1132e6ac/148c5e2e-2d42-4944-9524-d6f8f44422c9"
           (reference "U6")
           (unit 1)))))
@@
     (on_board yes)
     (dnp no)
-    (property "Reference" "C13"
+    (property "Reference" "C15"
       (at 706.12 29.37 0)
       (effects
@@
     (instances
       (project "prog"
-        (path "/730f52e2-cd0f-4a48-866b-cc2c9ca510b4/d40f7c6c-10f9-4e55-bf54-58eac98e1c03"
-          (reference "C13")
+        (path "/3a034faf-f518-4ff2-b4c3-d71a1132e6ac/148c5e2e-2d42-4944-9524-d6f8f44422c9"
+          (reference "C15")
           (unit 1)))))
   (global_label "+3V3"
@@
     (on_board yes)
     (dnp no)
-    (property "Reference" "C14"
+    (property "Reference" "C16"
       (at 55.88 115.73 0)
       (effects
@@
     (instances
       (project "prog"
-        (path "/730f52e2-cd0f-4a48-866b-cc2c9ca510b4/d40f7c6c-10f9-4e55-bf54-58eac98e1c03"
-          (reference "C14")
+        (path "/3a034faf-f518-4ff2-b4c3-d71a1132e6ac/148c5e2e-2d42-4944-9524-d6f8f44422c9"
+          (reference "C16")
           (unit 1)))))
   (global_label "+3V3"
@@
     (instances
       (project "prog"
-        (path "/730f52e2-cd0f-4a48-866b-cc2c9ca510b4/d40f7c6c-10f9-4e55-bf54-58eac98e1c03"
+        (path "/3a034faf-f518-4ff2-b4c3-d71a1132e6ac/148c5e2e-2d42-4944-9524-d6f8f44422c9"
           (reference "U7")
           (unit 1)))))
@@
     (on_board yes)
     (dnp no)
-    (property "Reference" "C15"
+    (property "Reference" "C17"
       (at 190.5 115.73 0)
       (effects
@@
     (instances
       (project "prog"
-        (path "/730f52e2-cd0f-4a48-866b-cc2c9ca510b4/d40f7c6c-10f9-4e55-bf54-58eac98e1c03"
-          (reference "C15")
+        (path "/3a034faf-f518-4ff2-b4c3-d71a1132e6ac/148c5e2e-2d42-4944-9524-d6f8f44422c9"
+          (reference "C17")
           (unit 1)))))
   (global_label "+3V3"
@@
     (on_board yes)
     (dnp no)
-    (property "Reference" "C16"
+    (property "Reference" "C18"
       (at 246.38 115.73 0)
       (effects
@@
     (instances
       (project "prog"
-        (path "/730f52e2-cd0f-4a48-866b-cc2c9ca510b4/d40f7c6c-10f9-4e55-bf54-58eac98e1c03"
-          (reference "C16")
+        (path "/3a034faf-f518-4ff2-b4c3-d71a1132e6ac/148c5e2e-2d42-4944-9524-d6f8f44422c9"
+          (reference "C18")
           (unit 1)))))
   (global_label "+3V3"
@@
     (instances
       (project "prog"
-        (path "/730f52e2-cd0f-4a48-866b-cc2c9ca510b4/d40f7c6c-10f9-4e55-bf54-58eac98e1c03"
+        (path "/3a034faf-f518-4ff2-b4c3-d71a1132e6ac/148c5e2e-2d42-4944-9524-d6f8f44422c9"
           (reference "U8")
           (unit 1)))))
@@
     (instances
       (project "prog"
-        (path "/730f52e2-cd0f-4a48-866b-cc2c9ca510b4/d40f7c6c-10f9-4e55-bf54-58eac98e1c03"
+        (path "/3a034faf-f518-4ff2-b4c3-d71a1132e6ac/148c5e2e-2d42-4944-9524-d6f8f44422c9"
           (reference "U8")
           (unit 2)))))
@@
     (instances
       (project "prog"
-        (path "/730f52e2-cd0f-4a48-866b-cc2c9ca510b4/d40f7c6c-10f9-4e55-bf54-58eac98e1c03"
+        (path "/3a034faf-f518-4ff2-b4c3-d71a1132e6ac/148c5e2e-2d42-4944-9524-d6f8f44422c9"
           (reference "U8")
           (unit 3)))))
@@
     (instances
       (project "prog"
-        (path "/730f52e2-cd0f-4a48-866b-cc2c9ca510b4/d40f7c6c-10f9-4e55-bf54-58eac98e1c03"
+        (path "/3a034faf-f518-4ff2-b4c3-d71a1132e6ac/148c5e2e-2d42-4944-9524-d6f8f44422c9"
           (reference "U8")
           (unit 4)))))
@@
     (instances
       (project "prog"
-        (path "/730f52e2-cd0f-4a48-866b-cc2c9ca510b4/d40f7c6c-10f9-4e55-bf54-58eac98e1c03"
+        (path "/3a034faf-f518-4ff2-b4c3-d71a1132e6ac/148c5e2e-2d42-4944-9524-d6f8f44422c9"
           (reference "U8")
           (unit 5)))))
@@
     (on_board yes)
     (dnp no)
-    (property "Reference" "C17"
+    (property "Reference" "C19"
       (at 637.54 115.73 0)
       (effects
@@
     (instances
       (project "prog"
-        (path "/730f52e2-cd0f-4a48-866b-cc2c9ca510b4/d40f7c6c-10f9-4e55-bf54-58eac98e1c03"
-          (reference "C17")
+        (path "/3a034faf-f518-4ff2-b4c3-d71a1132e6ac/148c5e2e-2d42-4944-9524-d6f8f44422c9"
+          (reference "C19")
           (unit 1)))))
   (global_label "+5V"
@@
     (instances
       (project "prog"
-        (path "/730f52e2-cd0f-4a48-866b-cc2c9ca510b4/d40f7c6c-10f9-4e55-bf54-58eac98e1c03"
+        (path "/3a034faf-f518-4ff2-b4c3-d71a1132e6ac/148c5e2e-2d42-4944-9524-d6f8f44422c9"
           (reference "U9")
           (unit 1)))))
@@
     (on_board yes)
     (dnp no)
-    (property "Reference" "C18"
+    (property "Reference" "C20"
       (at 55.88 202.09 0)
       (effects
@@
     (instances
       (project "prog"
-        (path "/730f52e2-cd0f-4a48-866b-cc2c9ca510b4/d40f7c6c-10f9-4e55-bf54-58eac98e1c03"
-          (reference "C18")
+        (path "/3a034faf-f518-4ff2-b4c3-d71a1132e6ac/148c5e2e-2d42-4944-9524-d6f8f44422c9"
+          (reference "C20")
           (unit 1)))))
   (global_label "+3V3"
@@
     (instances
       (project "prog"
-        (path "/730f52e2-cd0f-4a48-866b-cc2c9ca510b4/d40f7c6c-10f9-4e55-bf54-58eac98e1c03"
+        (path "/3a034faf-f518-4ff2-b4c3-d71a1132e6ac/148c5e2e-2d42-4944-9524-d6f8f44422c9"
           (reference "R8")
           (unit 1)))))
@@
     (instances
       (project "prog"
-        (path "/730f52e2-cd0f-4a48-866b-cc2c9ca510b4/d40f7c6c-10f9-4e55-bf54-58eac98e1c03"
+        (path "/3a034faf-f518-4ff2-b4c3-d71a1132e6ac/148c5e2e-2d42-4944-9524-d6f8f44422c9"
           (reference "R9")
           (unit 1)))))
