File: hardware/kicad/prog/fpga_v.kicad_sch (KiCad schematic)
At the start: 28 parts, among them J4 CONF V, U12 iCE40HX4K-TQ144, X2 25 MHz 3,3 V

Commit message: Régulateur 3,3 V à découpage, horloge SDRAM adaptée côté FPGA, U8 en 74AHCT125
- AP63203 (TSOT-23-6, sortie fixe 3,3 V, ~90 %) à la place de
  l'AMS1117 : ~0,15 W de pertes au lieu de ~0,75 W et moins de courant
  tiré sur le 5 V de la console ; L 4,7 µH, Cin 10 µF, Cout 2 x 22 µF.
- Résistance série de 33 ohms de l'horloge SDRAM déclarée avec le FPGA :
  placée à 2,7 mm de sa broche (au lieu de ~30 mm, côté SDRAM).
- CHA : U8 (16244 pour 2 canaux) remplacé par un 74AHCT125.
Cartes replacées, contrôle Freerouting sans violation ; routage des
deux cartes et vérification de timing en cours.

Co-Authored-By: Claude Opus 5.5 <noreply@anthropic.com>
Claude-Session: https://claude.ai/code/session_01WKfXP1YJ8otGxZ5dsY6Agh
Parts:
- removed C47, C48: 100n, Capacitor_SMD:C_0603_1608Metric, symbol Device:C
- added C67, C68: 100n, Capacitor_SMD:C_0603_1608Metric, symbol Device:C
- added R19: 470, Resistor_SMD:R_0603_1608Metric, symbol Device:R
- C51, C61, C62: value 10u -> 100n; footprint Capacitor_SMD:C_0805_2012Metric -> Capacitor_SMD:C_0603_1608Metric
- C53, C63, C66: value 100n -> 10u; footprint Capacitor_SMD:C_0603_1608Metric -> Capacitor_SMD:C_0805_2012Metric
- R18: value 470 -> 33
Connections:
- net +1V2: now also C52.1, C53.1
- net +3V3: now also C62.1, C63.1, C68.1; no longer C52.1, C53.1, C66.1
- net GND: now also C67.2, C68.2
- net V_LED: now also U12.84 (IOR_120), R19.1; no longer R18.1, U12.87 (IOR_136)
- net V_LED_K: now also R19.2; no longer R18.2
- net V_SD_A0: now also U12.3 (IOL_3A); no longer U12.4 (IOL_3B)
- net V_SD_A1: now also U12.4 (IOL_3B); no longer U12.7 (IOL_4A)
- net V_SD_A10: now also U12.2 (IOL_2B); no longer U12.3 (IOL_3A)
- net V_SD_A11: now also U12.110 (IOT_168); no longer U12.112 (IOT_169)
- net V_SD_A12: now also U12.112 (IOT_169); no longer U12.113 (IOT_170)
- net V_SD_A2: now also U12.7 (IOL_4A); no longer U12.8 (IOL_4B)
- net V_SD_A3: now also U12.8 (IOL_4B); no longer U12.9 (IOL_5A)
- net V_SD_A4: now also U12.101 (IOR_160); no longer U12.102 (IOR_161)
- net V_SD_A5: now also U12.102 (IOR_161); no longer U12.104 (IOR_164)
- net V_SD_A6: now also U12.104 (IOR_164); no longer U12.105 (IOR_165)
- net V_SD_A7: now also U12.105 (IOR_165); no longer U12.106 (IOR_166)
- net V_SD_A8: now also U12.106 (IOR_166); no longer U12.107 (IOR_167)
- net V_SD_A9: now also U12.107 (IOR_167); no longer U12.110 (IOT_168)
- net V_SD_BA0: now also U12.144 (IOT_222); no longer U12.1 (IOL_2A)
- net V_SD_BA1: now also U12.1 (IOL_2A); no longer U12.2 (IOL_2B)
- net V_SD_CAS_N: now also U12.141 (IOT_219); no longer U12.142 (IOT_220)
- net V_SD_CKE: now also U12.113 (IOT_170); no longer U12.114 (IOT_171)
- net V_SD_CLK: now also R18.1, U12.96 (IOR_146); no longer U12.101 (IOR_160)
- net V_SD_CS_N: now also U12.143 (IOT_221); no longer U12.144 (IOT_222)
- net V_SD_DQ0: now also U12.124 (IOT_191); no longer U12.125 (IOT_192)
- net V_SD_DQ1: now also U12.125 (IOT_192); no longer U12.128 (IOT_197_GBIN1)
- net V_SD_DQ10: now also U12.117 (IOT_174); no longer U12.118 (IOT_177)
- net V_SD_DQ11: now also U12.118 (IOT_177); no longer U12.119 (IOT_178)
- net V_SD_DQ12: now also U12.119 (IOT_178); no longer U12.120 (IOT_179)
- net V_SD_DQ13: now also U12.120 (IOT_179); no longer U12.121 (IOT_181)
- net V_SD_DQ14: now also U12.121 (IOT_181); no longer U12.122 (IOT_190)
- net V_SD_DQ15: now also U12.122 (IOT_190); no longer U12.124 (IOT_191)
- net V_SD_DQ2: now also U12.128 (IOT_197_GBIN1); no longer U12.130 (IOT_206)
- net V_SD_DQ3: now also U12.130 (IOT_206); no longer U12.134 (IOT_212)
- net V_SD_DQ4: now also U12.134 (IOT_212); no longer U12.135 (IOT_213)
- net V_SD_DQ5: now also U12.135 (IOT_213); no longer U12.136 (IOT_214)
- net V_SD_DQ6: now also U12.136 (IOT_214); no longer U12.137 (IOT_215)
- net V_SD_DQ7: now also U12.137 (IOT_215); no longer U12.138 (IOT_216)
- net V_SD_DQ8: now also U12.115 (IOT_172); no longer U12.116 (IOT_173)
- net V_SD_DQ9: now also U12.116 (IOT_173); no longer U12.117 (IOT_174)
- net V_SD_DQM0: now also U12.138 (IOT_216); no longer U12.139 (IOT_217)
- net V_SD_DQM1: now also U12.114 (IOT_171); no longer U12.115 (IOT_172)
- net V_SD_RAS_N: now also U12.142 (IOT_220); no longer U12.143 (IOT_221)
- net V_SD_WE_N: now also U12.139 (IOT_217); no longer U12.141 (IOT_219)
- net V_VCCPLL0: now also C64.1, C65.1; no longer C62.1, C63.1
- net V_VCCPLL1: now also C66.1, C67.1; no longer C64.1, C65.1
- new net V_SD_CLK_R: R18.2
