File: hardware/kicad/prog/prog.kicad_sch (KiCad schematic)
At the start: 0 parts

Commit message: Pico 2, microSD et bouton sur la carte PROG ; pistes d'alimentation larges
- La carte PROG est côté avant de la cartouche, composants vers l'avant :
  lecteur microSD et bouton accessibles. Le câble PROG-CHA porte
  désormais le bus de liaison C/SM ; connecteur au même endroit sur les
  deux cartes (x = 172 mm), prêt pour un connecteur carte à carte.
- Sous le Pico : ni piste ni via sur la face composants (pastilles de
  test nues sous le module).
- Classes de réseaux écrites dans le .kicad_pro : +5V et VSYS en 0,5 mm,
  +1V2 en 0,3 mm.
- Broches des FPGA réoptimisées ; contrôle Freerouting sans violation ;
  routage des deux cartes et vérification de timing en cours.

Co-Authored-By: Claude Opus 5.5 <noreply@anthropic.com>
Claude-Session: https://claude.ai/code/session_01WKfXP1YJ8otGxZ5dsY6Agh
Other:
- added sheet RP2350, carte SD, bouton (mcu.kicad_sch)
Changed lines of the file:
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@@
     (instances
       (project "prog"
-        (path "/da9dbc37-1614-4aa0-819a-d60fb574ce37"
+        (path "/730f52e2-cd0f-4a48-866b-cc2c9ca510b4"
           (page "2")))))
   (sheet
@@
     (instances
       (project "prog"
-        (path "/da9dbc37-1614-4aa0-819a-d60fb574ce37"
+        (path "/730f52e2-cd0f-4a48-866b-cc2c9ca510b4"
           (page "3")))))
   (sheet
@@
     (instances
       (project "prog"
-        (path "/da9dbc37-1614-4aa0-819a-d60fb574ce37"
+        (path "/730f52e2-cd0f-4a48-866b-cc2c9ca510b4"
           (page "4")))))
   (sheet
@@
     (instances
       (project "prog"
-        (path "/da9dbc37-1614-4aa0-819a-d60fb574ce37"
+        (path "/730f52e2-cd0f-4a48-866b-cc2c9ca510b4"
           (page "5")))))
   (sheet
@@
     (instances
       (project "prog"
-        (path "/da9dbc37-1614-4aa0-819a-d60fb574ce37"
+        (path "/730f52e2-cd0f-4a48-866b-cc2c9ca510b4"
           (page "6")))))
   (sheet
@@
     (instances
       (project "prog"
-        (path "/da9dbc37-1614-4aa0-819a-d60fb574ce37"
+        (path "/730f52e2-cd0f-4a48-866b-cc2c9ca510b4"
           (page "7")))))
+  (sheet
+    (at 152.4 68.58)
+    (size 50.8 25.4)
+    (fields_autoplaced)
+    (stroke
+      (width 0.1524)
+      (type solid))
+    (fill
+      (color 0 0 0 0.0000))
+    (property "Sheetname" "RP2350, carte SD, bouton"
+      (at 152.4 67.88 0)
+      (effects
+        (font
+          (size 1.27 1.27))
+        (justify left bottom)))
+    (property "Sheetfile" "mcu.kicad_sch"
+      (at 152.4 94.58 0)
+      (effects
+        (font
+          (size 1.27 1.27))
+        (justify left top) hide))
+    (instances
+      (project "prog"
+        (path "/730f52e2-cd0f-4a48-866b-cc2c9ca510b4"
+          (page "8")))))
   (sheet_instances
     (path "/"
