File: hardware/kicad/prog/sdram_p.kicad_sch (KiCad schematic)
At the start: 10 parts, among them U12 W9825G6KH-6

Commit message: FPGA configurés par le RP2350 depuis la carte SD (plus de flash)
- Matériel : flash SPI retirées (4 W25Q32, 12 résistances, 4
  condensateurs). Le bus de liaison arrive sur les broches de
  configuration des iCE40 (LK_SCK -> 70 SCK, LK_IO[0] -> 68 SDI,
  LK_CS_N -> 71 SS), qui redeviennent ces entrées après le démarrage.
  CRESET_N commun aux 4 FPGA, tiré à la masse, piloté par le RP2350
  (GP28) ; câble PROG-CHA en 2 x 7 (CRESET_N + masse). Connecteur 2 x 3
  de secours par FPGA (iceprog -S).
- Firmware : fpga_boot.c (reset commun en mode SPI esclave, envoi des
  SDAES/fpga_*.bin l'un après l'autre, contrôle de CDONE) ; testé sur
  PC (bitstreams reçus à l'identique, FPGA laissés en reset si un
  fichier manque).
- make -C hdl sd : fichiers à copier sur la carte SD.
- PCB : table de placement et références des FPGA mises à jour,
  broches réoptimisées.
Placement-routage des FPGA avec les nouvelles broches : en cours.

Co-Authored-By: Claude Opus 5.5 <noreply@anthropic.com>
Claude-Session: https://claude.ai/code/session_01WKfXP1YJ8otGxZ5dsY6Agh
Parts:
- removed C47: 10u, Capacitor_SMD:C_0805_2012Metric, symbol Device:C
- removed R17: 33, Resistor_SMD:R_0603_1608Metric, symbol Device:R
- removed U12: W9825G6KH-6, Package_SO:TSOP-II-54_22.2x10.16mm_P0.8mm, symbol Memory_RAM:MT48LC16M16A2TG
- added C39: 100n, Capacitor_SMD:C_0603_1608Metric, symbol Device:C
- added R14: 33, Resistor_SMD:R_0603_1608Metric, symbol Device:R
- added U11: W9825G6KH-6, Package_SO:TSOP-II-54_22.2x10.16mm_P0.8mm, symbol Memory_RAM:MT48LC16M16A2TG
- C46: value 100n -> 10u; footprint Capacitor_SMD:C_0603_1608Metric -> Capacitor_SMD:C_0805_2012Metric
Connections:
- net +3V3: now also C39.1, U11.1 (VDD), U11.14 (VDD), U11.27 (VDD), U11.3 (VDDQ), U11.43 (VDDQ), U11.49 (VDDQ), U11.9 (VDDQ)
- net GND: now also C39.2, U11.12 (VSSQ), U11.28 (VSS), U11.41 (VSS), U11.46 (VSSQ), U11.52 (VSSQ), U11.54 (VSS), U11.6 (VSSQ)
- net P_SD_A0: now also U11.23 (A0)
- net P_SD_A1: now also U11.24 (A1)
- net P_SD_A10: now also U11.22 (A10)
- net P_SD_A11: now also U11.35 (A11)
- net P_SD_A12: now also U11.36 (A12)
- net P_SD_A2: now also U11.25 (A2)
- net P_SD_A3: now also U11.26 (A3)
- net P_SD_A4: now also U11.29 (A4)
- net P_SD_A5: now also U11.30 (A5)
- net P_SD_A6: now also U11.31 (A6)
- net P_SD_A7: now also U11.32 (A7)
- net P_SD_A8: now also U11.33 (A8)
- net P_SD_A9: now also U11.34 (A9)
- net P_SD_BA0: now also U11.20 (BA0)
- net P_SD_BA1: now also U11.21 (BA1)
- net P_SD_CAS_N: now also U11.17 (~{CAS})
- net P_SD_CKE: now also U11.37 (CKE)
- net P_SD_CLK: now also R14.1
- net P_SD_CLK_R: now also R14.2, U11.38 (CLK)
- net P_SD_CS_N: now also U11.19 (~{CS})
- net P_SD_DQ0: now also U11.2 (DQ0)
- net P_SD_DQ1: now also U11.4 (DQ1)
- net P_SD_DQ10: now also U11.45 (DQ10)
- net P_SD_DQ11: now also U11.47 (DQ11)
- net P_SD_DQ12: now also U11.48 (DQ12)
- net P_SD_DQ13: now also U11.50 (DQ13)
- net P_SD_DQ14: now also U11.51 (DQ14)
- net P_SD_DQ15: now also U11.53 (DQ15)
- net P_SD_DQ2: now also U11.5 (DQ2)
- net P_SD_DQ3: now also U11.7 (DQ3)
- net P_SD_DQ4: now also U11.8 (DQ4)
- net P_SD_DQ5: now also U11.10 (DQ5)
- net P_SD_DQ6: now also U11.11 (DQ6)
- net P_SD_DQ7: now also U11.13 (DQ7)
- net P_SD_DQ8: now also U11.42 (DQ8)
- net P_SD_DQ9: now also U11.44 (DQ9)
- net P_SD_DQM0: now also U11.15 (DQML)
- net P_SD_DQM1: now also U11.39 (DQMH)
- net P_SD_RAS_N: now also U11.18 (~{RAS})
- net P_SD_WE_N: now also U11.16 (~{WE})
Changed lines of the file:
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@@
     (on_board yes)
     (dnp no)
-    (property "Reference" "U12"
+    (property "Reference" "U11"
       (at 68.58 28.1 0)
       (effects
@@
     (instances
       (project "prog"
-        (path "/a2c04eda-906b-4407-9534-e4dc8a098a56/c0b781c6-386c-4e12-8848-396807029a6f"
-          (reference "U12")
+        (path "/773ca91f-e149-4bba-abf7-6085382b056a/8740fb18-971a-44c1-bb08-7bc4fc34146f"
+          (reference "U11")
           (unit 1)))))
   (global_label "+3V3"
@@
     (on_board yes)
     (dnp no)
-    (property "Reference" "R17"
+    (property "Reference" "R14"
       (at 134.62 29.37 0)
       (effects
@@
     (instances
       (project "prog"
-        (path "/a2c04eda-906b-4407-9534-e4dc8a098a56/c0b781c6-386c-4e12-8848-396807029a6f"
-          (reference "R17")
+        (path "/773ca91f-e149-4bba-abf7-6085382b056a/8740fb18-971a-44c1-bb08-7bc4fc34146f"
+          (reference "R14")
           (unit 1)))))
   (global_label "P_SD_CLK"
@@
     (on_board yes)
     (dnp no)
-    (property "Reference" "C40"
+    (property "Reference" "C39"
       (at 190.5 29.37 0)
       (effects
@@
     (instances
       (project "prog"
-        (path "/a2c04eda-906b-4407-9534-e4dc8a098a56/c0b781c6-386c-4e12-8848-396807029a6f"
-          (reference "C40")
+        (path "/773ca91f-e149-4bba-abf7-6085382b056a/8740fb18-971a-44c1-bb08-7bc4fc34146f"
+          (reference "C39")
           (unit 1)))))
   (global_label "+3V3"
@@
     (on_board yes)
     (dnp no)
-    (property "Reference" "C41"
+    (property "Reference" "C40"
       (at 246.38 29.37 0)
       (effects
@@
     (instances
       (project "prog"
-        (path "/a2c04eda-906b-4407-9534-e4dc8a098a56/c0b781c6-386c-4e12-8848-396807029a6f"
-          (reference "C41")
+        (path "/773ca91f-e149-4bba-abf7-6085382b056a/8740fb18-971a-44c1-bb08-7bc4fc34146f"
+          (reference "C40")
           (unit 1)))))
   (global_label "+3V3"
@@
     (on_board yes)
     (dnp no)
-    (property "Reference" "C42"
+    (property "Reference" "C41"
       (at 299.72 29.37 0)
       (effects
@@
     (instances
       (project "prog"
-        (path "/a2c04eda-906b-4407-9534-e4dc8a098a56/c0b781c6-386c-4e12-8848-396807029a6f"
-          (reference "C42")
+        (path "/773ca91f-e149-4bba-abf7-6085382b056a/8740fb18-971a-44c1-bb08-7bc4fc34146f"
+          (reference "C41")
           (unit 1)))))
   (global_label "+3V3"
@@
     (on_board yes)
     (dnp no)
-    (property "Reference" "C43"
+    (property "Reference" "C42"
       (at 355.6 29.37 0)
       (effects
@@
     (instances
       (project "prog"
-        (path "/a2c04eda-906b-4407-9534-e4dc8a098a56/c0b781c6-386c-4e12-8848-396807029a6f"
-          (reference "C43")
+        (path "/773ca91f-e149-4bba-abf7-6085382b056a/8740fb18-971a-44c1-bb08-7bc4fc34146f"
+          (reference "C42")
           (unit 1)))))
   (global_label "+3V3"
@@
     (on_board yes)
     (dnp no)
-    (property "Reference" "C44"
+    (property "Reference" "C43"
       (at 411.48 29.37 0)
       (effects
@@
     (instances
       (project "prog"
-        (path "/a2c04eda-906b-4407-9534-e4dc8a098a56/c0b781c6-386c-4e12-8848-396807029a6f"
-          (reference "C44")
+        (path "/773ca91f-e149-4bba-abf7-6085382b056a/8740fb18-971a-44c1-bb08-7bc4fc34146f"
+          (reference "C43")
           (unit 1)))))
   (global_label "+3V3"
@@
     (on_board yes)
     (dnp no)
-    (property "Reference" "C45"
+    (property "Reference" "C44"
       (at 464.82 29.37 0)
       (effects
@@
     (instances
       (project "prog"
-        (path "/a2c04eda-906b-4407-9534-e4dc8a098a56/c0b781c6-386c-4e12-8848-396807029a6f"
-          (reference "C45")
+        (path "/773ca91f-e149-4bba-abf7-6085382b056a/8740fb18-971a-44c1-bb08-7bc4fc34146f"
+          (reference "C44")
           (unit 1)))))
   (global_label "+3V3"
@@
     (on_board yes)
     (dnp no)
-    (property "Reference" "C46"
+    (property "Reference" "C45"
       (at 520.7 29.37 0)
       (effects
@@
     (instances
       (project "prog"
-        (path "/a2c04eda-906b-4407-9534-e4dc8a098a56/c0b781c6-386c-4e12-8848-396807029a6f"
-          (reference "C46")
+        (path "/773ca91f-e149-4bba-abf7-6085382b056a/8740fb18-971a-44c1-bb08-7bc4fc34146f"
+          (reference "C45")
           (unit 1)))))
   (global_label "+3V3"
@@
     (on_board yes)
     (dnp no)
-    (property "Reference" "C47"
+    (property "Reference" "C46"
       (at 576.58 29.37 0)
       (effects
@@
     (instances
       (project "prog"
-        (path "/a2c04eda-906b-4407-9534-e4dc8a098a56/c0b781c6-386c-4e12-8848-396807029a6f"
-          (reference "C47")
+        (path "/773ca91f-e149-4bba-abf7-6085382b056a/8740fb18-971a-44c1-bb08-7bc4fc34146f"
+          (reference "C46")
           (unit 1)))))
   (global_label "+3V3"

Commit message: Régulateur 3,3 V à découpage, horloge SDRAM adaptée côté FPGA, U8 en 74AHCT125
- AP63203 (TSOT-23-6, sortie fixe 3,3 V, ~90 %) à la place de
  l'AMS1117 : ~0,15 W de pertes au lieu de ~0,75 W et moins de courant
  tiré sur le 5 V de la console ; L 4,7 µH, Cin 10 µF, Cout 2 x 22 µF.
- Résistance série de 33 ohms de l'horloge SDRAM déclarée avec le FPGA :
  placée à 2,7 mm de sa broche (au lieu de ~30 mm, côté SDRAM).
- CHA : U8 (16244 pour 2 canaux) remplacé par un 74AHCT125.
Cartes replacées, contrôle Freerouting sans violation ; routage des
deux cartes et vérification de timing en cours.

Co-Authored-By: Claude Opus 5.5 <noreply@anthropic.com>
Claude-Session: https://claude.ai/code/session_01WKfXP1YJ8otGxZ5dsY6Agh
Parts:
- removed C39, C40: 100n, Capacitor_SMD:C_0603_1608Metric, symbol Device:C
- removed R14: 33, Resistor_SMD:R_0603_1608Metric, symbol Device:R
- added C47: 100n, Capacitor_SMD:C_0603_1608Metric, symbol Device:C
- added C48: 10u, Capacitor_SMD:C_0805_2012Metric, symbol Device:C
- C46: value 10u -> 100n; footprint Capacitor_SMD:C_0805_2012Metric -> Capacitor_SMD:C_0603_1608Metric
Connections:
- net +3V3: now also C47.1, C48.1
- net GND: now also C47.2, C48.2
Changed lines of the file:
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@@
     (instances
       (project "prog"
-        (path "/730f52e2-cd0f-4a48-866b-cc2c9ca510b4/9883d523-be04-4a25-8c65-90da28f3a013"
+        (path "/3a034faf-f518-4ff2-b4c3-d71a1132e6ac/6970c1ac-40a6-4239-bf2e-bdf0f6d90e1b"
           (reference "U11")
           (unit 1)))))
@@
           (size 1.27 1.27)) hide)))
   (symbol
-    (lib_id "Device:R")
+    (lib_id "Device:C")
     (at 134.62 43.18 0)
     (unit 1)
@@
     (on_board yes)
     (dnp no)
-    (property "Reference" "R14"
+    (property "Reference" "C41"
       (at 134.62 29.37 0)
       (effects
         (font
           (size 1.27 1.27))))
-    (property "Value" "33"
+    (property "Value" "100n"
       (at 134.62 56.99 0)
       (effects
         (font
           (size 1.27 1.27))))
-    (property "Footprint" "Resistor_SMD:R_0603_1608Metric"
+    (property "Footprint" "Capacitor_SMD:C_0603_1608Metric"
       (at 134.62 43.18 0)
       (effects
@@
     (instances
       (project "prog"
-        (path "/730f52e2-cd0f-4a48-866b-cc2c9ca510b4/9883d523-be04-4a25-8c65-90da28f3a013"
-          (reference "R14")
+        (path "/3a034faf-f518-4ff2-b4c3-d71a1132e6ac/6970c1ac-40a6-4239-bf2e-bdf0f6d90e1b"
+          (reference "C41")
           (unit 1)))))
-  (global_label "P_SD_CLK"
+  (global_label "+3V3"
     (shape passive)
     (at 134.62 39.37 90)
@@
         (font
           (size 1.27 1.27)) hide)))
-  (global_label "P_SD_CLK_R"
+  (global_label "GND"
     (shape passive)
     (at 134.62 46.99 270)
@@
     (on_board yes)
     (dnp no)
-    (property "Reference" "C39"
+    (property "Reference" "C42"
       (at 190.5 29.37 0)
       (effects
@@
     (instances
       (project "prog"
-        (path "/730f52e2-cd0f-4a48-866b-cc2c9ca510b4/9883d523-be04-4a25-8c65-90da28f3a013"
-          (reference "C39")
+        (path "/3a034faf-f518-4ff2-b4c3-d71a1132e6ac/6970c1ac-40a6-4239-bf2e-bdf0f6d90e1b"
+          (reference "C42")
           (unit 1)))))
   (global_label "+3V3"
@@
     (on_board yes)
     (dnp no)
-    (property "Reference" "C40"
+    (property "Reference" "C43"
       (at 246.38 29.37 0)
       (effects
@@
     (instances
       (project "prog"
-        (path "/730f52e2-cd0f-4a48-866b-cc2c9ca510b4/9883d523-be04-4a25-8c65-90da28f3a013"
-          (reference "C40")
+        (path "/3a034faf-f518-4ff2-b4c3-d71a1132e6ac/6970c1ac-40a6-4239-bf2e-bdf0f6d90e1b"
+          (reference "C43")
           (unit 1)))))
   (global_label "+3V3"
@@
     (on_board yes)
     (dnp no)
-    (property "Reference" "C41"
+    (property "Reference" "C44"
       (at 299.72 29.37 0)
       (effects
@@
     (instances
       (project "prog"
-        (path "/730f52e2-cd0f-4a48-866b-cc2c9ca510b4/9883d523-be04-4a25-8c65-90da28f3a013"
-          (reference "C41")
+        (path "/3a034faf-f518-4ff2-b4c3-d71a1132e6ac/6970c1ac-40a6-4239-bf2e-bdf0f6d90e1b"
+          (reference "C44")
           (unit 1)))))
   (global_label "+3V3"
@@
     (on_board yes)
     (dnp no)
-    (property "Reference" "C42"
+    (property "Reference" "C45"
       (at 355.6 29.37 0)
       (effects
@@
     (instances
       (project "prog"
-        (path "/730f52e2-cd0f-4a48-866b-cc2c9ca510b4/9883d523-be04-4a25-8c65-90da28f3a013"
-          (reference "C42")
+        (path "/3a034faf-f518-4ff2-b4c3-d71a1132e6ac/6970c1ac-40a6-4239-bf2e-bdf0f6d90e1b"
+          (reference "C45")
           (unit 1)))))
   (global_label "+3V3"
@@
     (on_board yes)
     (dnp no)
-    (property "Reference" "C43"
+    (property "Reference" "C46"
       (at 411.48 29.37 0)
       (effects
@@
     (instances
       (project "prog"
-        (path "/730f52e2-cd0f-4a48-866b-cc2c9ca510b4/9883d523-be04-4a25-8c65-90da28f3a013"
-          (reference "C43")
+        (path "/3a034faf-f518-4ff2-b4c3-d71a1132e6ac/6970c1ac-40a6-4239-bf2e-bdf0f6d90e1b"
+          (reference "C46")
           (unit 1)))))
   (global_label "+3V3"
@@
     (on_board yes)
     (dnp no)
-    (property "Reference" "C44"
+    (property "Reference" "C47"
       (at 464.82 29.37 0)
       (effects
@@
     (instances
       (project "prog"
-        (path "/730f52e2-cd0f-4a48-866b-cc2c9ca510b4/9883d523-be04-4a25-8c65-90da28f3a013"
-          (reference "C44")
+        (path "/3a034faf-f518-4ff2-b4c3-d71a1132e6ac/6970c1ac-40a6-4239-bf2e-bdf0f6d90e1b"
+          (reference "C47")
           (unit 1)))))
   (global_label "+3V3"
@@
     (on_board yes)
     (dnp no)
-    (property "Reference" "C45"
+    (property "Reference" "C48"
       (at 520.7 29.37 0)
       (effects
         (font
           (size 1.27 1.27))))
-    (property "Value" "100n"
+    (property "Value" "10u"
       (at 520.7 56.99 0)
       (effects
         (font
           (size 1.27 1.27))))
-    (property "Footprint" "Capacitor_SMD:C_0603_1608Metric"
+    (property "Footprint" "Capacitor_SMD:C_0805_2012Metric"
       (at 520.7 43.18 0)
       (effects
@@
     (instances
       (project "prog"
-        (path "/730f52e2-cd0f-4a48-866b-cc2c9ca510b4/9883d523-be04-4a25-8c65-90da28f3a013"
-          (reference "C45")
+        (path "/3a034faf-f518-4ff2-b4c3-d71a1132e6ac/6970c1ac-40a6-4239-bf2e-bdf0f6d90e1b"
+          (reference "C48")
           (unit 1)))))
   (global_label "+3V3"
@@
       (effects
         (font
-          (size 1.27 1.27)) hide)))
-  (symbol
-    (lib_id "Device:C")
-    (at 576.58 43.18 0)
-    (unit 1)
-    (in_bom yes)
-    (on_board yes)
-    (dnp no)
-    (property "Reference" "C46"
-      (at 576.58 29.37 0)
-      (effects
-        (font
-          (size 1.27 1.27))))
-    (property "Value" "10u"
-      (at 576.58 56.99 0)
-      (effects
-        (font
-          (size 1.27 1.27))))
-    (property "Footprint" "Capacitor_SMD:C_0805_2012Metric"
-      (at 576.58 43.18 0)
-      (effects
-        (font
-          (size 1.27 1.27)) hide))
-    (property "Datasheet" "~"
-      (at 576.58 43.18 0)
-      (effects
-        (font
-          (size 1.27 1.27)) hide))
-    (pin "1"
-)
-    (pin "2"
-)
-    (instances
-      (project "prog"
-        (path "/730f52e2-cd0f-4a48-866b-cc2c9ca510b4/9883d523-be04-4a25-8c65-90da28f3a013"
-          (reference "C46")
-          (unit 1)))))
-  (global_label "+3V3"
-    (shape passive)
-    (at 576.58 39.37 90)
-    (fields_autoplaced)
-    (effects
-      (font
-        (size 1.27 1.27))
-      (justify left))
-    (property "Intersheetrefs" "${INTERSHEET_REFS}"
-      (at 576.58 39.37 0)
-      (effects
-        (font
-          (size 1.27 1.27)) hide)))
-  (global_label "GND"
-    (shape passive)
-    (at 576.58 46.99 270)
-    (fields_autoplaced)
-    (effects
-      (font
-        (size 1.27 1.27))
-      (justify right))
-    (property "Intersheetrefs" "${INTERSHEET_REFS}"
-      (at 576.58 46.99 0)
-      (effects
-        (font
