File: hardware/kicad/prog/sdram_v.kicad_sch (KiCad schematic)
At the start: 10 parts, among them U15 W9825G6KH-6

Commit message: FPGA configurés par le RP2350 depuis la carte SD (plus de flash)
- Matériel : flash SPI retirées (4 W25Q32, 12 résistances, 4
  condensateurs). Le bus de liaison arrive sur les broches de
  configuration des iCE40 (LK_SCK -> 70 SCK, LK_IO[0] -> 68 SDI,
  LK_CS_N -> 71 SS), qui redeviennent ces entrées après le démarrage.
  CRESET_N commun aux 4 FPGA, tiré à la masse, piloté par le RP2350
  (GP28) ; câble PROG-CHA en 2 x 7 (CRESET_N + masse). Connecteur 2 x 3
  de secours par FPGA (iceprog -S).
- Firmware : fpga_boot.c (reset commun en mode SPI esclave, envoi des
  SDAES/fpga_*.bin l'un après l'autre, contrôle de CDONE) ; testé sur
  PC (bitstreams reçus à l'identique, FPGA laissés en reset si un
  fichier manque).
- make -C hdl sd : fichiers à copier sur la carte SD.
- PCB : table de placement et références des FPGA mises à jour,
  broches réoptimisées.
Placement-routage des FPGA avec les nouvelles broches : en cours.

Co-Authored-By: Claude Opus 5.5 <noreply@anthropic.com>
Claude-Session: https://claude.ai/code/session_01WKfXP1YJ8otGxZ5dsY6Agh
Parts:
- removed C75: 100n, Capacitor_SMD:C_0603_1608Metric, symbol Device:C
- removed C76: 10u, Capacitor_SMD:C_0805_2012Metric, symbol Device:C
- removed R25: 33, Resistor_SMD:R_0603_1608Metric, symbol Device:R
- removed U15: W9825G6KH-6, Package_SO:TSOP-II-54_22.2x10.16mm_P0.8mm, symbol Memory_RAM:MT48LC16M16A2TG
- added C67, C68: 100n, Capacitor_SMD:C_0603_1608Metric, symbol Device:C
- added R19: 33, Resistor_SMD:R_0603_1608Metric, symbol Device:R
- added U13: W9825G6KH-6, Package_SO:TSOP-II-54_22.2x10.16mm_P0.8mm, symbol Memory_RAM:MT48LC16M16A2TG
- C74: value 100n -> 10u; footprint Capacitor_SMD:C_0603_1608Metric -> Capacitor_SMD:C_0805_2012Metric
Connections:
- net +3V3: now also C67.1, C68.1, U13.1 (VDD), U13.14 (VDD), U13.27 (VDD), U13.3 (VDDQ), U13.43 (VDDQ), U13.49 (VDDQ), U13.9 (VDDQ)
- net GND: now also C67.2, C68.2, U13.12 (VSSQ), U13.28 (VSS), U13.41 (VSS), U13.46 (VSSQ), U13.52 (VSSQ), U13.54 (VSS), U13.6 (VSSQ)
- net V_SD_A0: now also U13.23 (A0)
- net V_SD_A1: now also U13.24 (A1)
- net V_SD_A10: now also U13.22 (A10)
- net V_SD_A11: now also U13.35 (A11)
- net V_SD_A12: now also U13.36 (A12)
- net V_SD_A2: now also U13.25 (A2)
- net V_SD_A3: now also U13.26 (A3)
- net V_SD_A4: now also U13.29 (A4)
- net V_SD_A5: now also U13.30 (A5)
- net V_SD_A6: now also U13.31 (A6)
- net V_SD_A7: now also U13.32 (A7)
- net V_SD_A8: now also U13.33 (A8)
- net V_SD_A9: now also U13.34 (A9)
- net V_SD_BA0: now also U13.20 (BA0)
- net V_SD_BA1: now also U13.21 (BA1)
- net V_SD_CAS_N: now also U13.17 (~{CAS})
- net V_SD_CKE: now also U13.37 (CKE)
- net V_SD_CLK: now also R19.1
- net V_SD_CLK_R: now also R19.2, U13.38 (CLK)
- net V_SD_CS_N: now also U13.19 (~{CS})
- net V_SD_DQ0: now also U13.2 (DQ0)
- net V_SD_DQ1: now also U13.4 (DQ1)
- net V_SD_DQ10: now also U13.45 (DQ10)
- net V_SD_DQ11: now also U13.47 (DQ11)
- net V_SD_DQ12: now also U13.48 (DQ12)
- net V_SD_DQ13: now also U13.50 (DQ13)
- net V_SD_DQ14: now also U13.51 (DQ14)
- net V_SD_DQ15: now also U13.53 (DQ15)
- net V_SD_DQ2: now also U13.5 (DQ2)
- net V_SD_DQ3: now also U13.7 (DQ3)
- net V_SD_DQ4: now also U13.8 (DQ4)
- net V_SD_DQ5: now also U13.10 (DQ5)
- net V_SD_DQ6: now also U13.11 (DQ6)
- net V_SD_DQ7: now also U13.13 (DQ7)
- net V_SD_DQ8: now also U13.42 (DQ8)
- net V_SD_DQ9: now also U13.44 (DQ9)
- net V_SD_DQM0: now also U13.15 (DQML)
- net V_SD_DQM1: now also U13.39 (DQMH)
- net V_SD_RAS_N: now also U13.18 (~{RAS})
- net V_SD_WE_N: now also U13.16 (~{WE})
Changed lines of the file:
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@@
     (on_board yes)
     (dnp no)
-    (property "Reference" "U15"
+    (property "Reference" "U13"
       (at 68.58 28.1 0)
       (effects
@@
     (instances
       (project "prog"
-        (path "/a2c04eda-906b-4407-9534-e4dc8a098a56/17027125-807e-465f-9b8e-373a957a00ab"
-          (reference "U15")
+        (path "/773ca91f-e149-4bba-abf7-6085382b056a/ae3e0653-9471-4df5-9bf8-7b65d62bc753"
+          (reference "U13")
           (unit 1)))))
   (global_label "+3V3"
@@
     (on_board yes)
     (dnp no)
-    (property "Reference" "R25"
+    (property "Reference" "R19"
       (at 134.62 29.37 0)
       (effects
@@
     (instances
       (project "prog"
-        (path "/a2c04eda-906b-4407-9534-e4dc8a098a56/17027125-807e-465f-9b8e-373a957a00ab"
-          (reference "R25")
+        (path "/773ca91f-e149-4bba-abf7-6085382b056a/ae3e0653-9471-4df5-9bf8-7b65d62bc753"
+          (reference "R19")
           (unit 1)))))
   (global_label "V_SD_CLK"
@@
     (on_board yes)
     (dnp no)
-    (property "Reference" "C69"
+    (property "Reference" "C67"
       (at 190.5 29.37 0)
       (effects
@@
     (instances
       (project "prog"
-        (path "/a2c04eda-906b-4407-9534-e4dc8a098a56/17027125-807e-465f-9b8e-373a957a00ab"
-          (reference "C69")
+        (path "/773ca91f-e149-4bba-abf7-6085382b056a/ae3e0653-9471-4df5-9bf8-7b65d62bc753"
+          (reference "C67")
           (unit 1)))))
   (global_label "+3V3"
@@
     (on_board yes)
     (dnp no)
-    (property "Reference" "C70"
+    (property "Reference" "C68"
       (at 246.38 29.37 0)
       (effects
@@
     (instances
       (project "prog"
-        (path "/a2c04eda-906b-4407-9534-e4dc8a098a56/17027125-807e-465f-9b8e-373a957a00ab"
-          (reference "C70")
+        (path "/773ca91f-e149-4bba-abf7-6085382b056a/ae3e0653-9471-4df5-9bf8-7b65d62bc753"
+          (reference "C68")
           (unit 1)))))
   (global_label "+3V3"
@@
     (on_board yes)
     (dnp no)
-    (property "Reference" "C71"
+    (property "Reference" "C69"
       (at 299.72 29.37 0)
       (effects
@@
     (instances
       (project "prog"
-        (path "/a2c04eda-906b-4407-9534-e4dc8a098a56/17027125-807e-465f-9b8e-373a957a00ab"
-          (reference "C71")
+        (path "/773ca91f-e149-4bba-abf7-6085382b056a/ae3e0653-9471-4df5-9bf8-7b65d62bc753"
+          (reference "C69")
           (unit 1)))))
   (global_label "+3V3"
@@
     (on_board yes)
     (dnp no)
-    (property "Reference" "C72"
+    (property "Reference" "C70"
       (at 355.6 29.37 0)
       (effects
@@
     (instances
       (project "prog"
-        (path "/a2c04eda-906b-4407-9534-e4dc8a098a56/17027125-807e-465f-9b8e-373a957a00ab"
-          (reference "C72")
+        (path "/773ca91f-e149-4bba-abf7-6085382b056a/ae3e0653-9471-4df5-9bf8-7b65d62bc753"
+          (reference "C70")
           (unit 1)))))
   (global_label "+3V3"
@@
     (on_board yes)
     (dnp no)
-    (property "Reference" "C73"
+    (property "Reference" "C71"
       (at 411.48 29.37 0)
       (effects
@@
     (instances
       (project "prog"
-        (path "/a2c04eda-906b-4407-9534-e4dc8a098a56/17027125-807e-465f-9b8e-373a957a00ab"
-          (reference "C73")
+        (path "/773ca91f-e149-4bba-abf7-6085382b056a/ae3e0653-9471-4df5-9bf8-7b65d62bc753"
+          (reference "C71")
           (unit 1)))))
   (global_label "+3V3"
@@
     (on_board yes)
     (dnp no)
-    (property "Reference" "C74"
+    (property "Reference" "C72"
       (at 464.82 29.37 0)
       (effects
@@
     (instances
       (project "prog"
-        (path "/a2c04eda-906b-4407-9534-e4dc8a098a56/17027125-807e-465f-9b8e-373a957a00ab"
-          (reference "C74")
+        (path "/773ca91f-e149-4bba-abf7-6085382b056a/ae3e0653-9471-4df5-9bf8-7b65d62bc753"
+          (reference "C72")
           (unit 1)))))
   (global_label "+3V3"
@@
     (on_board yes)
     (dnp no)
-    (property "Reference" "C75"
+    (property "Reference" "C73"
       (at 520.7 29.37 0)
       (effects
@@
     (instances
       (project "prog"
-        (path "/a2c04eda-906b-4407-9534-e4dc8a098a56/17027125-807e-465f-9b8e-373a957a00ab"
-          (reference "C75")
+        (path "/773ca91f-e149-4bba-abf7-6085382b056a/ae3e0653-9471-4df5-9bf8-7b65d62bc753"
+          (reference "C73")
           (unit 1)))))
   (global_label "+3V3"
@@
     (on_board yes)
     (dnp no)
-    (property "Reference" "C76"
+    (property "Reference" "C74"
       (at 576.58 29.37 0)
       (effects
@@
     (instances
       (project "prog"
-        (path "/a2c04eda-906b-4407-9534-e4dc8a098a56/17027125-807e-465f-9b8e-373a957a00ab"
-          (reference "C76")
+        (path "/773ca91f-e149-4bba-abf7-6085382b056a/ae3e0653-9471-4df5-9bf8-7b65d62bc753"
+          (reference "C74")
           (unit 1)))))
   (global_label "+3V3"

Commit message: Régulateur 3,3 V à découpage, horloge SDRAM adaptée côté FPGA, U8 en 74AHCT125
- AP63203 (TSOT-23-6, sortie fixe 3,3 V, ~90 %) à la place de
  l'AMS1117 : ~0,15 W de pertes au lieu de ~0,75 W et moins de courant
  tiré sur le 5 V de la console ; L 4,7 µH, Cin 10 µF, Cout 2 x 22 µF.
- Résistance série de 33 ohms de l'horloge SDRAM déclarée avec le FPGA :
  placée à 2,7 mm de sa broche (au lieu de ~30 mm, côté SDRAM).
- CHA : U8 (16244 pour 2 canaux) remplacé par un 74AHCT125.
Cartes replacées, contrôle Freerouting sans violation ; routage des
deux cartes et vérification de timing en cours.

Co-Authored-By: Claude Opus 5.5 <noreply@anthropic.com>
Claude-Session: https://claude.ai/code/session_01WKfXP1YJ8otGxZ5dsY6Agh
Parts:
- removed C67, C68: 100n, Capacitor_SMD:C_0603_1608Metric, symbol Device:C
- removed R19: 33, Resistor_SMD:R_0603_1608Metric, symbol Device:R
- added C75: 100n, Capacitor_SMD:C_0603_1608Metric, symbol Device:C
- added C76: 10u, Capacitor_SMD:C_0805_2012Metric, symbol Device:C
- C74: value 10u -> 100n; footprint Capacitor_SMD:C_0805_2012Metric -> Capacitor_SMD:C_0603_1608Metric
Connections:
- net +3V3: now also C75.1, C76.1
- net GND: now also C75.2, C76.2
Changed lines of the file:
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@@
     (instances
       (project "prog"
-        (path "/730f52e2-cd0f-4a48-866b-cc2c9ca510b4/e0b64567-bdf6-4a1e-887a-de3a9f80cf9f"
+        (path "/3a034faf-f518-4ff2-b4c3-d71a1132e6ac/fbd40e6d-9067-4b9e-b588-537a90cb836c"
           (reference "U13")
           (unit 1)))))
@@
           (size 1.27 1.27)) hide)))
   (symbol
-    (lib_id "Device:R")
+    (lib_id "Device:C")
     (at 134.62 43.18 0)
     (unit 1)
@@
     (on_board yes)
     (dnp no)
-    (property "Reference" "R19"
+    (property "Reference" "C69"
       (at 134.62 29.37 0)
       (effects
         (font
           (size 1.27 1.27))))
-    (property "Value" "33"
+    (property "Value" "100n"
       (at 134.62 56.99 0)
       (effects
         (font
           (size 1.27 1.27))))
-    (property "Footprint" "Resistor_SMD:R_0603_1608Metric"
+    (property "Footprint" "Capacitor_SMD:C_0603_1608Metric"
       (at 134.62 43.18 0)
       (effects
@@
     (instances
       (project "prog"
-        (path "/730f52e2-cd0f-4a48-866b-cc2c9ca510b4/e0b64567-bdf6-4a1e-887a-de3a9f80cf9f"
-          (reference "R19")
+        (path "/3a034faf-f518-4ff2-b4c3-d71a1132e6ac/fbd40e6d-9067-4b9e-b588-537a90cb836c"
+          (reference "C69")
           (unit 1)))))
-  (global_label "V_SD_CLK"
+  (global_label "+3V3"
     (shape passive)
     (at 134.62 39.37 90)
@@
         (font
           (size 1.27 1.27)) hide)))
-  (global_label "V_SD_CLK_R"
+  (global_label "GND"
     (shape passive)
     (at 134.62 46.99 270)
@@
     (on_board yes)
     (dnp no)
-    (property "Reference" "C67"
+    (property "Reference" "C70"
       (at 190.5 29.37 0)
       (effects
@@
     (instances
       (project "prog"
-        (path "/730f52e2-cd0f-4a48-866b-cc2c9ca510b4/e0b64567-bdf6-4a1e-887a-de3a9f80cf9f"
-          (reference "C67")
+        (path "/3a034faf-f518-4ff2-b4c3-d71a1132e6ac/fbd40e6d-9067-4b9e-b588-537a90cb836c"
+          (reference "C70")
           (unit 1)))))
   (global_label "+3V3"
@@
     (on_board yes)
     (dnp no)
-    (property "Reference" "C68"
+    (property "Reference" "C71"
       (at 246.38 29.37 0)
       (effects
@@
     (instances
       (project "prog"
-        (path "/730f52e2-cd0f-4a48-866b-cc2c9ca510b4/e0b64567-bdf6-4a1e-887a-de3a9f80cf9f"
-          (reference "C68")
+        (path "/3a034faf-f518-4ff2-b4c3-d71a1132e6ac/fbd40e6d-9067-4b9e-b588-537a90cb836c"
+          (reference "C71")
           (unit 1)))))
   (global_label "+3V3"
@@
     (on_board yes)
     (dnp no)
-    (property "Reference" "C69"
+    (property "Reference" "C72"
       (at 299.72 29.37 0)
       (effects
@@
     (instances
       (project "prog"
-        (path "/730f52e2-cd0f-4a48-866b-cc2c9ca510b4/e0b64567-bdf6-4a1e-887a-de3a9f80cf9f"
-          (reference "C69")
+        (path "/3a034faf-f518-4ff2-b4c3-d71a1132e6ac/fbd40e6d-9067-4b9e-b588-537a90cb836c"
+          (reference "C72")
           (unit 1)))))
   (global_label "+3V3"
@@
     (on_board yes)
     (dnp no)
-    (property "Reference" "C70"
+    (property "Reference" "C73"
       (at 355.6 29.37 0)
       (effects
@@
     (instances
       (project "prog"
-        (path "/730f52e2-cd0f-4a48-866b-cc2c9ca510b4/e0b64567-bdf6-4a1e-887a-de3a9f80cf9f"
-          (reference "C70")
+        (path "/3a034faf-f518-4ff2-b4c3-d71a1132e6ac/fbd40e6d-9067-4b9e-b588-537a90cb836c"
+          (reference "C73")
           (unit 1)))))
   (global_label "+3V3"
@@
     (on_board yes)
     (dnp no)
-    (property "Reference" "C71"
+    (property "Reference" "C74"
       (at 411.48 29.37 0)
       (effects
@@
     (instances
       (project "prog"
-        (path "/730f52e2-cd0f-4a48-866b-cc2c9ca510b4/e0b64567-bdf6-4a1e-887a-de3a9f80cf9f"
-          (reference "C71")
+        (path "/3a034faf-f518-4ff2-b4c3-d71a1132e6ac/fbd40e6d-9067-4b9e-b588-537a90cb836c"
+          (reference "C74")
           (unit 1)))))
   (global_label "+3V3"
@@
     (on_board yes)
     (dnp no)
-    (property "Reference" "C72"
+    (property "Reference" "C75"
       (at 464.82 29.37 0)
       (effects
@@
     (instances
       (project "prog"
-        (path "/730f52e2-cd0f-4a48-866b-cc2c9ca510b4/e0b64567-bdf6-4a1e-887a-de3a9f80cf9f"
-          (reference "C72")
+        (path "/3a034faf-f518-4ff2-b4c3-d71a1132e6ac/fbd40e6d-9067-4b9e-b588-537a90cb836c"
+          (reference "C75")
           (unit 1)))))
   (global_label "+3V3"
@@
     (on_board yes)
     (dnp no)
-    (property "Reference" "C73"
+    (property "Reference" "C76"
       (at 520.7 29.37 0)
       (effects
         (font
           (size 1.27 1.27))))
-    (property "Value" "100n"
+    (property "Value" "10u"
       (at 520.7 56.99 0)
       (effects
         (font
           (size 1.27 1.27))))
-    (property "Footprint" "Capacitor_SMD:C_0603_1608Metric"
+    (property "Footprint" "Capacitor_SMD:C_0805_2012Metric"
       (at 520.7 43.18 0)
       (effects
@@
     (instances
       (project "prog"
-        (path "/730f52e2-cd0f-4a48-866b-cc2c9ca510b4/e0b64567-bdf6-4a1e-887a-de3a9f80cf9f"
-          (reference "C73")
+        (path "/3a034faf-f518-4ff2-b4c3-d71a1132e6ac/fbd40e6d-9067-4b9e-b588-537a90cb836c"
+          (reference "C76")
           (unit 1)))))
   (global_label "+3V3"
@@
       (effects
         (font
-          (size 1.27 1.27)) hide)))
-  (symbol
-    (lib_id "Device:C")
-    (at 576.58 43.18 0)
-    (unit 1)
-    (in_bom yes)
-    (on_board yes)
-    (dnp no)
-    (property "Reference" "C74"
-      (at 576.58 29.37 0)
-      (effects
-        (font
-          (size 1.27 1.27))))
-    (property "Value" "10u"
-      (at 576.58 56.99 0)
-      (effects
-        (font
-          (size 1.27 1.27))))
-    (property "Footprint" "Capacitor_SMD:C_0805_2012Metric"
-      (at 576.58 43.18 0)
-      (effects
-        (font
-          (size 1.27 1.27)) hide))
-    (property "Datasheet" "~"
-      (at 576.58 43.18 0)
-      (effects
-        (font
-          (size 1.27 1.27)) hide))
-    (pin "1"
-)
-    (pin "2"
-)
-    (instances
-      (project "prog"
-        (path "/730f52e2-cd0f-4a48-866b-cc2c9ca510b4/e0b64567-bdf6-4a1e-887a-de3a9f80cf9f"
-          (reference "C74")
-          (unit 1)))))
-  (global_label "+3V3"
-    (shape passive)
-    (at 576.58 39.37 90)
-    (fields_autoplaced)
-    (effects
-      (font
-        (size 1.27 1.27))
-      (justify left))
-    (property "Intersheetrefs" "${INTERSHEET_REFS}"
-      (at 576.58 39.37 0)
-      (effects
-        (font
-          (size 1.27 1.27)) hide)))
-  (global_label "GND"
-    (shape passive)
-    (at 576.58 46.99 270)
-    (fields_autoplaced)
-    (effects
-      (font
-        (size 1.27 1.27))
-      (justify right))
-    (property "Intersheetrefs" "${INTERSHEET_REFS}"
-      (at 576.58 46.99 0)
-      (effects
-        (font
